File: elec/layout/demomatrix/demomatrix.kicad_pcb (KiCad board)
At the start: 2 copper layers, 1 part

Commit message: pixel demos
Parts:
- removed R1: 10kΩ ±1% 100mW, UNI_ROYAL_0603WAF1002T5E:R0603
- added LED1: , TCWIN_TC5050RGBW4D06_4CJHR3_AFW421A:LED-SMD_8P-L5.0-W5.0-TL-FD, F.Cu at (5.20, 5.00)
- added U1: , ATOPILE_PIXEL:pixel, F.Cu at (0.00, 0.00)
Routing:
- net cathode_red: track 0.00 -> 8.84 mm, vias 0 -> 2
- net cathode_cold_white: track 0.00 -> 7.80 mm
- net anode: track 0.00 -> 7.36 mm
- net cathode_green: track 0.00 -> 6.96 mm, vias 0 -> 2
- net cathode_blue: track 0.00 -> 5.29 mm

Commit message: Pixel15 & Cluster
Parts:
- added LED10: , HONGLITRONIC_HL_5050RGBW_S1_A27:LED-SMD_8P-L5.0-W5.0-P1.20_HL-5050RGBW-S1-A27, F.Cu at (48.5, 50.9)
- added LED11: , HONGLITRONIC_HL_5050RGBW_S1_A27:LED-SMD_8P-L5.0-W5.0-P1.20_HL-5050RGBW-S1-A27, F.Cu at (54.3, 45.9)
- added LED12: , HONGLITRONIC_HL_5050RGBW_S1_A27:LED-SMD_8P-L5.0-W5.0-P1.20_HL-5050RGBW-S1-A27, F.Cu at (48.5, 45.9)
- added LED13: , HONGLITRONIC_HL_5050RGBW_S1_A27:LED-SMD_8P-L5.0-W5.0-P1.20_HL-5050RGBW-S1-A27, F.Cu at (38.7, 50.9)
- added LED14: , HONGLITRONIC_HL_5050RGBW_S1_A27:LED-SMD_8P-L5.0-W5.0-P1.20_HL-5050RGBW-S1-A27, F.Cu at (32.9, 50.9)
- added LED15: , HONGLITRONIC_HL_5050RGBW_S1_A27:LED-SMD_8P-L5.0-W5.0-P1.20_HL-5050RGBW-S1-A27, F.Cu at (38.7, 45.9)
- added LED16: , HONGLITRONIC_HL_5050RGBW_S1_A27:LED-SMD_8P-L5.0-W5.0-P1.20_HL-5050RGBW-S1-A27, F.Cu at (32.9, 45.9)
- added LED17: , HONGLITRONIC_HL_5050RGBW_S1_A27:LED-SMD_8P-L5.0-W5.0-P1.20_HL-5050RGBW-S1-A27, F.Cu at (74.6, 28.1)
- added LED18: , HONGLITRONIC_HL_5050RGBW_S1_A27:LED-SMD_8P-L5.0-W5.0-P1.20_HL-5050RGBW-S1-A27, F.Cu at (80.4, 28.1)
- added LED19: , HONGLITRONIC_HL_5050RGBW_S1_A27:LED-SMD_8P-L5.0-W5.0-P1.20_HL-5050RGBW-S1-A27, F.Cu at (74.6, 33.1)
- added LED2: , HONGLITRONIC_HL_5050RGBW_S1_A27:LED-SMD_8P-L5.0-W5.0-P1.20_HL-5050RGBW-S1-A27, F.Cu at (38.2, 28.1)
- added LED20: , HONGLITRONIC_HL_5050RGBW_S1_A27:LED-SMD_8P-L5.0-W5.0-P1.20_HL-5050RGBW-S1-A27, F.Cu at (80.4, 33.1)
- added LED21: , HONGLITRONIC_HL_5050RGBW_S1_A27:LED-SMD_8P-L5.0-W5.0-P1.20_HL-5050RGBW-S1-A27, F.Cu at (90.3, 28.1)
- added LED22: , HONGLITRONIC_HL_5050RGBW_S1_A27:LED-SMD_8P-L5.0-W5.0-P1.20_HL-5050RGBW-S1-A27, F.Cu at (96.1, 28.1)
- added LED23: , HONGLITRONIC_HL_5050RGBW_S1_A27:LED-SMD_8P-L5.0-W5.0-P1.20_HL-5050RGBW-S1-A27, F.Cu at (90.3, 33.1)
- added LED24: , HONGLITRONIC_HL_5050RGBW_S1_A27:LED-SMD_8P-L5.0-W5.0-P1.20_HL-5050RGBW-S1-A27, F.Cu at (96.1, 33.1)
- added LED25: , HONGLITRONIC_HL_5050RGBW_S1_A27:LED-SMD_8P-L5.0-W5.0-P1.20_HL-5050RGBW-S1-A27, F.Cu at (96.5, 50.9)
- added LED26: , HONGLITRONIC_HL_5050RGBW_S1_A27:LED-SMD_8P-L5.0-W5.0-P1.20_HL-5050RGBW-S1-A27, F.Cu at (90.7, 50.9)
- added LED27: , HONGLITRONIC_HL_5050RGBW_S1_A27:LED-SMD_8P-L5.0-W5.0-P1.20_HL-5050RGBW-S1-A27, F.Cu at (96.5, 45.9)
- added LED28: , HONGLITRONIC_HL_5050RGBW_S1_A27:LED-SMD_8P-L5.0-W5.0-P1.20_HL-5050RGBW-S1-A27, F.Cu at (90.7, 45.9)
- added LED29: , HONGLITRONIC_HL_5050RGBW_S1_A27:LED-SMD_8P-L5.0-W5.0-P1.20_HL-5050RGBW-S1-A27, F.Cu at (80.8, 50.9)
- added LED3: , HONGLITRONIC_HL_5050RGBW_S1_A27:LED-SMD_8P-L5.0-W5.0-P1.20_HL-5050RGBW-S1-A27, F.Cu at (32.4, 33.1)
- added LED30: , HONGLITRONIC_HL_5050RGBW_S1_A27:LED-SMD_8P-L5.0-W5.0-P1.20_HL-5050RGBW-S1-A27, F.Cu at (75.0, 50.9)
- added LED31: , HONGLITRONIC_HL_5050RGBW_S1_A27:LED-SMD_8P-L5.0-W5.0-P1.20_HL-5050RGBW-S1-A27, F.Cu at (80.8, 45.9)
- added LED32: , HONGLITRONIC_HL_5050RGBW_S1_A27:LED-SMD_8P-L5.0-W5.0-P1.20_HL-5050RGBW-S1-A27, F.Cu at (75.0, 45.9)
- added LED33: , HONGLITRONIC_HL_5050RGBW_S1_A27:LED-SMD_8P-L5.0-W5.0-P1.20_HL-5050RGBW-S1-A27, F.Cu at (116.5, 28.1)
- added LED34: , HONGLITRONIC_HL_5050RGBW_S1_A27:LED-SMD_8P-L5.0-W5.0-P1.20_HL-5050RGBW-S1-A27, F.Cu at (122.3, 28.1)
- added LED35: , HONGLITRONIC_HL_5050RGBW_S1_A27:LED-SMD_8P-L5.0-W5.0-P1.20_HL-5050RGBW-S1-A27, F.Cu at (116.5, 33.1)
- added LED36: , HONGLITRONIC_HL_5050RGBW_S1_A27:LED-SMD_8P-L5.0-W5.0-P1.20_HL-5050RGBW-S1-A27, F.Cu at (122.3, 33.1)
- added LED37: , HONGLITRONIC_HL_5050RGBW_S1_A27:LED-SMD_8P-L5.0-W5.0-P1.20_HL-5050RGBW-S1-A27, F.Cu at (132.2, 28.1)
- added LED38: , HONGLITRONIC_HL_5050RGBW_S1_A27:LED-SMD_8P-L5.0-W5.0-P1.20_HL-5050RGBW-S1-A27, F.Cu at (138.0, 28.1)
- added LED39: , HONGLITRONIC_HL_5050RGBW_S1_A27:LED-SMD_8P-L5.0-W5.0-P1.20_HL-5050RGBW-S1-A27, F.Cu at (132.2, 33.1)
- added LED4: , HONGLITRONIC_HL_5050RGBW_S1_A27:LED-SMD_8P-L5.0-W5.0-P1.20_HL-5050RGBW-S1-A27, F.Cu at (38.2, 33.1)
- added LED40: , HONGLITRONIC_HL_5050RGBW_S1_A27:LED-SMD_8P-L5.0-W5.0-P1.20_HL-5050RGBW-S1-A27, F.Cu at (138.0, 33.1)
- added LED41: , HONGLITRONIC_HL_5050RGBW_S1_A27:LED-SMD_8P-L5.0-W5.0-P1.20_HL-5050RGBW-S1-A27, F.Cu at (138.4, 50.9)
- added LED42: , HONGLITRONIC_HL_5050RGBW_S1_A27:LED-SMD_8P-L5.0-W5.0-P1.20_HL-5050RGBW-S1-A27, F.Cu at (132.6, 50.9)
- added LED43: , HONGLITRONIC_HL_5050RGBW_S1_A27:LED-SMD_8P-L5.0-W5.0-P1.20_HL-5050RGBW-S1-A27, F.Cu at (138.4, 45.9)
- added LED44: , HONGLITRONIC_HL_5050RGBW_S1_A27:LED-SMD_8P-L5.0-W5.0-P1.20_HL-5050RGBW-S1-A27, F.Cu at (132.6, 45.9)
- added LED45: , HONGLITRONIC_HL_5050RGBW_S1_A27:LED-SMD_8P-L5.0-W5.0-P1.20_HL-5050RGBW-S1-A27, F.Cu at (122.7, 50.9)
- added LED46: , HONGLITRONIC_HL_5050RGBW_S1_A27:LED-SMD_8P-L5.0-W5.0-P1.20_HL-5050RGBW-S1-A27, F.Cu at (116.9, 50.9)
- added LED47: , HONGLITRONIC_HL_5050RGBW_S1_A27:LED-SMD_8P-L5.0-W5.0-P1.20_HL-5050RGBW-S1-A27, F.Cu at (122.7, 45.9)
- added LED48: , HONGLITRONIC_HL_5050RGBW_S1_A27:LED-SMD_8P-L5.0-W5.0-P1.20_HL-5050RGBW-S1-A27, F.Cu at (116.9, 45.9)
- added LED49: , HONGLITRONIC_HL_5050RGBW_S1_A27:LED-SMD_8P-L5.0-W5.0-P1.20_HL-5050RGBW-S1-A27, F.Cu at (158.9, 28.1)
- added LED5: , HONGLITRONIC_HL_5050RGBW_S1_A27:LED-SMD_8P-L5.0-W5.0-P1.20_HL-5050RGBW-S1-A27, F.Cu at (48.1, 28.1)
- added LED50: , HONGLITRONIC_HL_5050RGBW_S1_A27:LED-SMD_8P-L5.0-W5.0-P1.20_HL-5050RGBW-S1-A27, F.Cu at (164.7, 28.1)
- added LED51: , HONGLITRONIC_HL_5050RGBW_S1_A27:LED-SMD_8P-L5.0-W5.0-P1.20_HL-5050RGBW-S1-A27, F.Cu at (158.9, 33.1)
- added LED52: , HONGLITRONIC_HL_5050RGBW_S1_A27:LED-SMD_8P-L5.0-W5.0-P1.20_HL-5050RGBW-S1-A27, F.Cu at (164.7, 33.1)
- added LED53: , HONGLITRONIC_HL_5050RGBW_S1_A27:LED-SMD_8P-L5.0-W5.0-P1.20_HL-5050RGBW-S1-A27, F.Cu at (174.6, 28.1)
- added LED54: , HONGLITRONIC_HL_5050RGBW_S1_A27:LED-SMD_8P-L5.0-W5.0-P1.20_HL-5050RGBW-S1-A27, F.Cu at (180.4, 28.1)
- added LED55: , HONGLITRONIC_HL_5050RGBW_S1_A27:LED-SMD_8P-L5.0-W5.0-P1.20_HL-5050RGBW-S1-A27, F.Cu at (174.6, 33.1)
- added LED56: , HONGLITRONIC_HL_5050RGBW_S1_A27:LED-SMD_8P-L5.0-W5.0-P1.20_HL-5050RGBW-S1-A27, F.Cu at (180.4, 33.1)
- added LED57: , HONGLITRONIC_HL_5050RGBW_S1_A27:LED-SMD_8P-L5.0-W5.0-P1.20_HL-5050RGBW-S1-A27, F.Cu at (180.8, 50.9)
- added LED58: , HONGLITRONIC_HL_5050RGBW_S1_A27:LED-SMD_8P-L5.0-W5.0-P1.20_HL-5050RGBW-S1-A27, F.Cu at (175.0, 50.9)
- added LED59: , HONGLITRONIC_HL_5050RGBW_S1_A27:LED-SMD_8P-L5.0-W5.0-P1.20_HL-5050RGBW-S1-A27, F.Cu at (180.8, 45.9)
- added LED6: , HONGLITRONIC_HL_5050RGBW_S1_A27:LED-SMD_8P-L5.0-W5.0-P1.20_HL-5050RGBW-S1-A27, F.Cu at (53.9, 28.1)
- added LED60: , HONGLITRONIC_HL_5050RGBW_S1_A27:LED-SMD_8P-L5.0-W5.0-P1.20_HL-5050RGBW-S1-A27, F.Cu at (175.0, 45.9)
- added LED61: , HONGLITRONIC_HL_5050RGBW_S1_A27:LED-SMD_8P-L5.0-W5.0-P1.20_HL-5050RGBW-S1-A27, F.Cu at (165.1, 50.9)
- added LED62: , HONGLITRONIC_HL_5050RGBW_S1_A27:LED-SMD_8P-L5.0-W5.0-P1.20_HL-5050RGBW-S1-A27, F.Cu at (159.3, 50.9)
- added LED63: , HONGLITRONIC_HL_5050RGBW_S1_A27:LED-SMD_8P-L5.0-W5.0-P1.20_HL-5050RGBW-S1-A27, F.Cu at (165.1, 45.9)
- added LED64: , HONGLITRONIC_HL_5050RGBW_S1_A27:LED-SMD_8P-L5.0-W5.0-P1.20_HL-5050RGBW-S1-A27, F.Cu at (159.3, 45.9)
- added LED7: , HONGLITRONIC_HL_5050RGBW_S1_A27:LED-SMD_8P-L5.0-W5.0-P1.20_HL-5050RGBW-S1-A27, F.Cu at (48.1, 33.1)
- added LED8: , HONGLITRONIC_HL_5050RGBW_S1_A27:LED-SMD_8P-L5.0-W5.0-P1.20_HL-5050RGBW-S1-A27, F.Cu at (53.9, 33.1)
- added LED9: , HONGLITRONIC_HL_5050RGBW_S1_A27:LED-SMD_8P-L5.0-W5.0-P1.20_HL-5050RGBW-S1-A27, F.Cu at (54.3, 50.9)
- added U10: , ATOPILE_PIXEL15:pixel15, F.Cu at (127.8, 24.1)
- added U11: , ATOPILE_PIXEL15:pixel15, F.Cu at (142.8, 54.9)
- added U12: , ATOPILE_PIXEL15:pixel15, F.Cu at (127.1, 54.9)
- added U13: , ATOPILE_PIXEL15:pixel15, F.Cu at (154.5, 24.1)
- added U14: , ATOPILE_PIXEL15:pixel15, F.Cu at (170.2, 24.1)
- added U15: , ATOPILE_PIXEL15:pixel15, F.Cu at (185.2, 54.9)
- added U16: , ATOPILE_PIXEL15:pixel15, F.Cu at (169.5, 54.9)
- added U2: , ATOPILE_PIXEL15:pixel15, F.Cu at (43.7, 24.1)
- added U3: , ATOPILE_PIXEL15:pixel15, F.Cu at (58.7, 54.9)
- added U4: , ATOPILE_PIXEL15:pixel15, F.Cu at (43.1, 54.9)
- added U5: , ATOPILE_PIXEL15:pixel15, F.Cu at (70.2, 24.1)
- added U6: , ATOPILE_PIXEL15:pixel15, F.Cu at (85.9, 24.1)
- added U7: , ATOPILE_PIXEL15:pixel15, F.Cu at (100.9, 54.9)
- added U8: , ATOPILE_PIXEL15:pixel15, F.Cu at (85.2, 54.9)
- added U9: , ATOPILE_PIXEL15:pixel15, F.Cu at (112.1, 24.1)
- LED1: footprint TCWIN_TC5050RGBW4D06_4CJHR3_AFW421A:LED-SMD_8P-L5.0-W5.0-TL-FD -> HONGLITRONIC_HL_5050RGBW_S1_A27:LED-SMD_8P-L5.0-W5.0-P1.20_HL-5050RGBW-S1-A27
- U1: footprint ATOPILE_PIXEL:pixel -> ATOPILE_PIXEL15:pixel15
- moved U1 37.0 mm to (28.0, 24.1)
- moved LED1 35.7 mm to (32.4, 28.1), turned to 180 degrees
Connections:
- net cathode_ir renamed clusters[0].rows[0].pixels[0]-cathode_ir
- net cathode_uv renamed clusters[0].rows[0].pixels[0]-cathode_uv
- net cathode_warm_white renamed clusters[0].rows[0].pixels[0]-cathode_warm_white
- LED1 pad 1: anode -> clusters[0].rows[0].pixels[0]-cathode_cold_white
- LED1 pad 2: anode -> clusters[0].rows[0].pixels[0]-anode
- LED1 pad 3: anode -> clusters[0].rows[0].pixels[0]-cathode_blue
- LED1 pad 4: anode -> clusters[0].rows[0].pixels[0]-anode
- LED1 pad 5: cathode_cold_white -> clusters[0].rows[0].pixels[0]-cathode_green
- LED1 pad 6: cathode_blue -> clusters[0].rows[0].pixels[0]-anode
- LED1 pad 7: cathode_green -> clusters[0].rows[0].pixels[0]-cathode_red
- LED1 pad 8: cathode_red -> clusters[0].rows[0].pixels[0]-anode
- U1 pad 1: anode -> clusters[0].rows[0].pixels[0]-anode
- U1 pad 2: cathode_red -> clusters[0].rows[0].pixels[0]-cathode_red
- U1 pad 3: cathode_green -> clusters[0].rows[0].pixels[0]-cathode_green
- U1 pad 4: cathode_blue -> clusters[0].rows[0].pixels[0]-cathode_blue
- U1 pad 6: cathode_cold_white -> clusters[0].rows[0].pixels[0]-cathode_cold_white
Routing:
- net clusters[2].rows[0].pixels[1]-cathode_blue: track 0.00 -> 36.2 mm, vias 0 -> 2
- net clusters[3].rows[0].pixels[0]-cathode_blue: track 0.00 -> 36.2 mm, vias 0 -> 2
- net clusters[2].rows[0].pixels[0]-cathode_blue: track 0.00 -> 36.2 mm, vias 0 -> 2
- net clusters[1].rows[1].pixels[1]-cathode_blue: track 0.00 -> 36.2 mm, vias 0 -> 2
- net clusters[1].rows[0].pixels[0]-cathode_blue: track 0.00 -> 36.2 mm, vias 0 -> 2
- net clusters[2].rows[1].pixels[1]-cathode_blue: track 0.00 -> 36.2 mm, vias 0 -> 2
- net clusters[2].rows[1].pixels[0]-cathode_blue: track 0.00 -> 36.2 mm, vias 0 -> 2
- net clusters[1].rows[0].pixels[1]-cathode_blue: track 0.00 -> 36.2 mm, vias 0 -> 2
- net clusters[0].rows[0].pixels[0]-cathode_blue: track 0.00 -> 36.2 mm, vias 0 -> 2
- net clusters[3].rows[0].pixels[1]-cathode_blue: track 0.00 -> 36.2 mm, vias 0 -> 2
- net clusters[0].rows[1].pixels[1]-cathode_blue: track 0.00 -> 36.2 mm, vias 0 -> 2
- net clusters[0].rows[1].pixels[0]-cathode_blue: track 0.00 -> 36.2 mm, vias 0 -> 2
- net clusters[0].rows[0].pixels[1]-cathode_blue: track 0.00 -> 36.2 mm, vias 0 -> 2
- net clusters[3].rows[1].pixels[1]-cathode_blue: track 0.00 -> 36.2 mm, vias 0 -> 2
- net clusters[3].rows[1].pixels[0]-cathode_blue: track 0.00 -> 36.2 mm, vias 0 -> 2
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