File: elec/layout/demomatrix/demomatrix.kicad_pcb (KiCad board)
At the start: 2 copper layers, 24.6 x 8.1 mm, 1592 parts

Commit message: column and panel layout
Parts:
- moved LOGO1 1155.6 mm to (1156.2, -29.8)
- moved U10 180.9 mm to (69.9, 35.0)
- moved U8 180.9 mm to (69.9, 20.0)
- moved C10 180.9 mm to (61.5, 28.4)
- moved C11 180.9 mm to (63.2, 26.7)
- moved C12 180.9 mm to (61.5, 41.7)
- moved C13 180.9 mm to (78.2, 28.3)
- moved C14 180.9 mm to (76.5, 43.4)
- moved C15 180.9 mm to (63.2, 43.4)
- moved C16 180.9 mm to (78.1, 41.7)
- moved C18 180.9 mm to (64.8, 35.0)
- moved LED17 180.9 mm to (58.7, 23.8)
- moved LED18 180.9 mm to (66.1, 23.8)
- moved LED19 180.9 mm to (66.1, 31.2)
- moved LED20 180.9 mm to (58.7, 31.2)
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Connections:
- USB1 pad : net -> (no net)
