File: elec/layout/pixel15tc5050/pixel15tc5050.kicad_pcb (KiCad board)
At the start: 2 copper layers, 5 parts

Commit message: updating rp2040
Connections:
- LED1 pad 1: anode -> rgbs[0]-anodes-anode
- LED1 pad 2: anode -> rgbs[0]-anodes-anode
- LED1 pad 3: anode -> rgbs[0]-anodes-anode
- LED1 pad 4: anode -> rgbs[0]-anodes-anode
- LED1 pad 5: cathode_cold_white -> rgbs[1]-anodes-anode-1
- LED1 pad 6: cathode_blue -> rgbs[1]-anodes-anode-0
- LED1 pad 7: cathode_green -> rgbs[1]-anodes-anode-2
- LED1 pad 8: cathode_red -> rgbs[1]-anodes-anode-3
- LED2 pad 1: anode -> rgbs[1]-anodes-anode-3
- LED2 pad 2: anode -> rgbs[1]-anodes-anode-2
- LED2 pad 3: anode -> rgbs[1]-anodes-anode-0
- LED2 pad 4: anode -> rgbs[1]-anodes-anode-1
- LED2 pad 5: cathode_cold_white -> rgbs[2]-anodes-anode-1
- LED2 pad 6: cathode_blue -> rgbs[2]-anodes-anode-0
- LED2 pad 7: cathode_green -> rgbs[2]-anodes-anode-2
- LED2 pad 8: cathode_red -> rgbs[2]-anodes-anode-3
- LED3 pad 1: anode -> rgbs[2]-anodes-anode-3
- LED3 pad 2: anode -> rgbs[2]-anodes-anode-2
- LED3 pad 3: anode -> rgbs[2]-anodes-anode-0
- LED3 pad 4: anode -> rgbs[2]-anodes-anode-1
- LED3 pad 5: cathode_cold_white -> rgbs[3]-anodes-anode-1
- LED3 pad 6: cathode_blue -> rgbs[3]-anodes-anode-0
- LED3 pad 7: cathode_green -> rgbs[3]-anodes-anode-2
- LED3 pad 8: cathode_red -> rgbs[3]-anodes-anode-3
- LED4 pad 1: anode -> rgbs[3]-anodes-anode-3
- LED4 pad 2: anode -> rgbs[3]-anodes-anode-2
- LED4 pad 3: anode -> rgbs[3]-anodes-anode-0
- LED4 pad 4: anode -> rgbs[3]-anodes-anode-1
- LED4 pad 5: cathode_cold_white -> rgbs[3]-cathodes-cathode-1
- LED4 pad 6: cathode_blue -> rgbs[3]-cathodes-cathode-0
- LED4 pad 7: cathode_green -> rgbs[3]-cathodes-cathode-2
- LED4 pad 8: cathode_red -> rgbs[3]-cathodes-cathode-3
