File: elec/layout/cluster2x2/cluster2x2.kicad_pcb (KiCad board)
At the start: 2 copper layers, 20 parts

Commit message: cluster with driver
Parts:
- added C1: 100nF ±10% 16V X7R, Samsung_Electro_Mechanics_CL05B104KO5NNNC:C0402, F.Cu at (-4.94, -10.0)
- added R1: 309Ω ±1% 62.5mW, VO_SCR0402F309R:R0402, F.Cu at (-6.04, -10.0)
- added U5: , MBI_MBI5043GP_A:SSOP-24_L8.8-W4.0-P0.64-LS6.2-BL, F.Cu at (0.00, -10.0)
- moved U3 74.9 mm to (0.00, 15.0), turned to 0 degrees
- moved LED9 63.8 mm to (3.80, 18.8), turned to 45 degrees
- moved LED10 53.0 mm to (11.2, 18.8), turned to -45 degrees
- moved LED12 52.9 mm to (3.80, 26.2), turned to 135 degrees
- moved U4 52.2 mm to (15.0, 15.0), turned to 0 degrees
- moved LED11 51.4 mm to (11.2, 26.2), turned to -135 degrees
- moved LED8 45.3 mm to (18.8, 11.2), turned to 135 degrees
- moved LED4 44.7 mm to (3.80, 11.2), turned to 135 degrees
- moved LED5 41.9 mm to (18.8, 3.80), turned to 45 degrees
- moved LED1 41.4 mm to (3.80, 3.80), turned to 45 degrees
- moved U2 41.3 mm to (15.0, 0.00)
- moved LED13 41.0 mm to (18.8, 18.8), turned to 45 degrees
- moved U1 40.8 mm to (0.00, 0.00)
- moved LED6 40.6 mm to (26.2, 3.80), turned to -45 degrees
- moved LED2 40.1 mm to (11.2, 3.80), turned to -45 degrees
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Connections:
- net rows[0].pixels[0]-cathode_ir renamed rows[0].pixels[0]-ir
- net rows[0].pixels[0]-cathode_uv renamed rows[0].pixels[0]-uv
- net rows[0].pixels[0]-cathode_warm_white renamed rows[0].pixels[0]-warm_white
- net rows[0].pixels[1]-cathode_ir renamed rows[0].pixels[1]-ir
- net rows[0].pixels[1]-cathode_uv renamed rows[0].pixels[1]-uv
- net rows[0].pixels[1]-cathode_warm_white renamed rows[0].pixels[1]-warm_white
- net rows[1].pixels[0]-cathode_ir renamed rows[1].pixels[0]-ir
- net rows[1].pixels[0]-cathode_uv renamed rows[1].pixels[0]-uv
- net rows[1].pixels[0]-cathode_warm_white renamed rows[1].pixels[0]-warm_white
- net rows[1].pixels[1]-cathode_ir renamed rows[1].pixels[1]-ir
- net rows[1].pixels[1]-cathode_uv renamed rows[1].pixels[1]-uv
- net rows[1].pixels[1]-cathode_warm_white renamed rows[1].pixels[1]-warm_white
- LED1 pad 1: rows[0].pixels[0]-cathode_cold_white -> rows[0].pixels[0]-cold_white-1
- LED1 pad 2: rows[0].pixels[0]-anode -> -anode
- LED1 pad 3: rows[0].pixels[0]-cathode_blue -> rows[0].pixels[0]-blue-1
- LED1 pad 4: rows[0].pixels[0]-anode -> -anode
- LED1 pad 5: rows[0].pixels[0]-cathode_green -> rows[0].pixels[0]-green-1
- LED1 pad 6: rows[0].pixels[0]-anode -> -anode
- LED1 pad 7: rows[0].pixels[0]-cathode_red -> rows[0].pixels[0]-red-0
- LED1 pad 8: rows[0].pixels[0]-anode -> -anode
- LED10 pad 1: rows[1].pixels[0]-cathode_cold_white -> rows[1].pixels[0]-cold_white-2
- LED10 pad 2: rows[1].pixels[0]-anode -> rows[1].pixels[0]-cold_white-1
- LED10 pad 3: rows[1].pixels[0]-cathode_blue -> rows[1].pixels[0]-blue-2
- LED10 pad 4: rows[1].pixels[0]-anode -> rows[1].pixels[0]-blue-1
- LED10 pad 5: rows[1].pixels[0]-cathode_green -> rows[1].pixels[0]-green-2
- LED10 pad 6: rows[1].pixels[0]-anode -> rows[1].pixels[0]-green-1
- LED10 pad 7: rows[1].pixels[0]-cathode_red -> rows[1].pixels[0]-red-2
- LED10 pad 8: rows[1].pixels[0]-anode -> rows[1].pixels[0]-red-1
- LED11 pad 1: rows[1].pixels[0]-cathode_cold_white -> rows[1].pixels[0]-cold_white-3
- LED11 pad 2: rows[1].pixels[0]-anode -> rows[1].pixels[0]-cold_white-2
- LED11 pad 3: rows[1].pixels[0]-cathode_blue -> rows[1].pixels[0]-blue-3
- LED11 pad 4: rows[1].pixels[0]-anode -> rows[1].pixels[0]-blue-2
- LED11 pad 5: rows[1].pixels[0]-cathode_green -> rows[1].pixels[0]-green-3
- LED11 pad 6: rows[1].pixels[0]-anode -> rows[1].pixels[0]-green-2
- LED11 pad 7: rows[1].pixels[0]-cathode_red -> rows[1].pixels[0]-red-3
- LED11 pad 8: rows[1].pixels[0]-anode -> rows[1].pixels[0]-red-2
- LED12 pad 1: rows[1].pixels[0]-cathode_cold_white -> rows[1].pixels[0]-cold_white-0
- LED12 pad 2: rows[1].pixels[0]-anode -> rows[1].pixels[0]-cold_white-3
- LED12 pad 3: rows[1].pixels[0]-cathode_blue -> rows[1].pixels[0]-blue-0
- LED12 pad 4: rows[1].pixels[0]-anode -> rows[1].pixels[0]-blue-3
- LED12 pad 5: rows[1].pixels[0]-cathode_green -> rows[1].pixels[0]-green-0
- LED12 pad 6: rows[1].pixels[0]-anode -> rows[1].pixels[0]-green-3
- LED12 pad 7: rows[1].pixels[0]-cathode_red -> rows[1].pixels[0]-red-0
- LED12 pad 8: rows[1].pixels[0]-anode -> rows[1].pixels[0]-red-3
- LED13 pad 1: rows[1].pixels[1]-cathode_cold_white -> rows[1].pixels[1]-cold_white-1
- LED13 pad 3: rows[1].pixels[1]-cathode_blue -> rows[1].pixels[1]-blue-1
- LED13 pad 5: rows[1].pixels[1]-cathode_green -> rows[1].pixels[1]-green-1
- LED13 pad 7: rows[1].pixels[1]-cathode_red -> rows[1].pixels[1]-red-1
- LED14 pad 1: rows[1].pixels[1]-cathode_cold_white -> rows[1].pixels[1]-cold_white-2
- LED14 pad 2: rows[1].pixels[1]-anode -> rows[1].pixels[1]-cold_white-1
- LED14 pad 3: rows[1].pixels[1]-cathode_blue -> rows[1].pixels[1]-blue-2
- LED14 pad 4: rows[1].pixels[1]-anode -> rows[1].pixels[1]-blue-1
- LED14 pad 5: rows[1].pixels[1]-cathode_green -> rows[1].pixels[1]-green-2
- LED14 pad 6: rows[1].pixels[1]-anode -> rows[1].pixels[1]-green-1
- LED14 pad 7: rows[1].pixels[1]-cathode_red -> rows[1].pixels[1]-red-2
- LED14 pad 8: rows[1].pixels[1]-anode -> rows[1].pixels[1]-red-1
- LED15 pad 1: rows[1].pixels[1]-cathode_cold_white -> rows[1].pixels[1]-cold_white-3
- LED15 pad 2: rows[1].pixels[1]-anode -> rows[1].pixels[1]-cold_white-2
- LED15 pad 3: rows[1].pixels[1]-cathode_blue -> rows[1].pixels[1]-blue-3
- LED15 pad 4: rows[1].pixels[1]-anode -> rows[1].pixels[1]-blue-2
- LED15 pad 5: rows[1].pixels[1]-cathode_green -> rows[1].pixels[1]-green-3
- LED15 pad 6: rows[1].pixels[1]-anode -> rows[1].pixels[1]-green-2
- LED15 pad 7: rows[1].pixels[1]-cathode_red -> rows[1].pixels[1]-red-3
- LED15 pad 8: rows[1].pixels[1]-anode -> rows[1].pixels[1]-red-2
- LED16 pad 1: rows[1].pixels[1]-cathode_cold_white -> rows[1].pixels[1]-cold_white-0
- LED16 pad 2: rows[1].pixels[1]-anode -> rows[1].pixels[1]-cold_white-3
- LED16 pad 3: rows[1].pixels[1]-cathode_blue -> rows[1].pixels[1]-blue-0
- LED16 pad 4: rows[1].pixels[1]-anode -> rows[1].pixels[1]-blue-3
- LED16 pad 5: rows[1].pixels[1]-cathode_green -> rows[1].pixels[1]-green-0
- LED16 pad 6: rows[1].pixels[1]-anode -> rows[1].pixels[1]-green-3
- LED16 pad 7: rows[1].pixels[1]-cathode_red -> rows[1].pixels[1]-red-0
- LED16 pad 8: rows[1].pixels[1]-anode -> rows[1].pixels[1]-red-3
- LED2 pad 1: rows[0].pixels[0]-cathode_cold_white -> rows[0].pixels[0]-cold_white-2
- LED2 pad 2: rows[0].pixels[0]-anode -> rows[0].pixels[0]-cold_white-1
- LED2 pad 3: rows[0].pixels[0]-cathode_blue -> rows[0].pixels[0]-blue-2
- LED2 pad 4: rows[0].pixels[0]-anode -> rows[0].pixels[0]-blue-1
- LED2 pad 5: rows[0].pixels[0]-cathode_green -> rows[0].pixels[0]-green-2
- LED2 pad 6: rows[0].pixels[0]-anode -> rows[0].pixels[0]-green-1
- LED2 pad 7: rows[0].pixels[0]-cathode_red -> rows[0].pixels[0]-red-1
- LED2 pad 8: rows[0].pixels[0]-anode -> rows[0].pixels[0]-red-0
- LED3 pad 1: rows[0].pixels[0]-cathode_cold_white -> rows[0].pixels[0]-cold_white-3
- LED3 pad 2: rows[0].pixels[0]-anode -> rows[0].pixels[0]-cold_white-2
- LED3 pad 3: rows[0].pixels[0]-cathode_blue -> rows[0].pixels[0]-blue-3
- LED3 pad 4: rows[0].pixels[0]-anode -> rows[0].pixels[0]-blue-2
- LED3 pad 5: rows[0].pixels[0]-cathode_green -> rows[0].pixels[0]-green-3
- LED3 pad 6: rows[0].pixels[0]-anode -> rows[0].pixels[0]-green-2
- LED3 pad 7: rows[0].pixels[0]-cathode_red -> rows[0].pixels[0]-red-2
- LED3 pad 8: rows[0].pixels[0]-anode -> rows[0].pixels[0]-red-1
- LED4 pad 1: rows[0].pixels[0]-cathode_cold_white -> rows[0].pixels[0]-cold_white-0
- LED4 pad 2: rows[0].pixels[0]-anode -> rows[0].pixels[0]-cold_white-3
- LED4 pad 3: rows[0].pixels[0]-cathode_blue -> rows[0].pixels[0]-blue-0
- LED4 pad 4: rows[0].pixels[0]-anode -> rows[0].pixels[0]-blue-3
- LED4 pad 5: rows[0].pixels[0]-cathode_green -> rows[0].pixels[0]-green-0
- LED4 pad 6: rows[0].pixels[0]-anode -> rows[0].pixels[0]-green-3
- LED4 pad 7: rows[0].pixels[0]-cathode_red -> -red
- LED4 pad 8: rows[0].pixels[0]-anode -> rows[0].pixels[0]-red-2
- LED5 pad 1: rows[0].pixels[1]-cathode_cold_white -> rows[0].pixels[1]-cold_white-1
- LED5 pad 3: rows[0].pixels[1]-cathode_blue -> rows[0].pixels[1]-blue-1
- LED5 pad 5: rows[0].pixels[1]-cathode_green -> rows[0].pixels[1]-green-1
- LED5 pad 7: rows[0].pixels[1]-cathode_red -> rows[0].pixels[1]-red-1
- LED6 pad 1: rows[0].pixels[1]-cathode_cold_white -> rows[0].pixels[1]-cold_white-2
- LED6 pad 2: rows[0].pixels[1]-anode -> rows[0].pixels[1]-cold_white-1
- LED6 pad 3: rows[0].pixels[1]-cathode_blue -> rows[0].pixels[1]-blue-2
- LED6 pad 4: rows[0].pixels[1]-anode -> rows[0].pixels[1]-blue-1
- LED6 pad 5: rows[0].pixels[1]-cathode_green -> rows[0].pixels[1]-green-2
- LED6 pad 6: rows[0].pixels[1]-anode -> rows[0].pixels[1]-green-1
- LED6 pad 7: rows[0].pixels[1]-cathode_red -> rows[0].pixels[1]-red-2
- LED6 pad 8: rows[0].pixels[1]-anode -> rows[0].pixels[1]-red-1
- LED7 pad 1: rows[0].pixels[1]-cathode_cold_white -> rows[0].pixels[1]-cold_white-3
- LED7 pad 2: rows[0].pixels[1]-anode -> rows[0].pixels[1]-cold_white-2
- LED7 pad 3: rows[0].pixels[1]-cathode_blue -> rows[0].pixels[1]-blue-3
- LED7 pad 4: rows[0].pixels[1]-anode -> rows[0].pixels[1]-blue-2
- LED7 pad 5: rows[0].pixels[1]-cathode_green -> rows[0].pixels[1]-green-3
- LED7 pad 6: rows[0].pixels[1]-anode -> rows[0].pixels[1]-green-2
- LED7 pad 7: rows[0].pixels[1]-cathode_red -> rows[0].pixels[1]-red-3
- LED7 pad 8: rows[0].pixels[1]-anode -> rows[0].pixels[1]-red-2
- LED8 pad 1: rows[0].pixels[1]-cathode_cold_white -> rows[0].pixels[1]-cold_white-0
- LED8 pad 2: rows[0].pixels[1]-anode -> rows[0].pixels[1]-cold_white-3
- LED8 pad 3: rows[0].pixels[1]-cathode_blue -> rows[0].pixels[1]-blue-0
- LED8 pad 4: rows[0].pixels[1]-anode -> rows[0].pixels[1]-blue-3
- LED8 pad 5: rows[0].pixels[1]-cathode_green -> rows[0].pixels[1]-green-0
- LED8 pad 6: rows[0].pixels[1]-anode -> rows[0].pixels[1]-green-3
- LED8 pad 7: rows[0].pixels[1]-cathode_red -> rows[0].pixels[1]-red-0
- LED8 pad 8: rows[0].pixels[1]-anode -> rows[0].pixels[1]-red-3
- LED9 pad 1: rows[1].pixels[0]-cathode_cold_white -> rows[1].pixels[0]-cold_white-1
- LED9 pad 3: rows[1].pixels[0]-cathode_blue -> rows[1].pixels[0]-blue-1
- LED9 pad 5: rows[1].pixels[0]-cathode_green -> rows[1].pixels[0]-green-1
- LED9 pad 7: rows[1].pixels[0]-cathode_red -> rows[1].pixels[0]-red-1
- U1 pad 1: rows[0].pixels[0]-anode -> -anode
- U1 pad 2: rows[0].pixels[0]-cathode_red -> -red
- U1 pad 3: rows[0].pixels[0]-cathode_green -> rows[0].pixels[0]-green-0
- U1 pad 4: rows[0].pixels[0]-cathode_blue -> rows[0].pixels[0]-blue-0
- U1 pad 6: rows[0].pixels[0]-cathode_cold_white -> rows[0].pixels[0]-cold_white-0
- U2 pad 2: rows[0].pixels[1]-cathode_red -> rows[0].pixels[1]-red-0
- U2 pad 3: rows[0].pixels[1]-cathode_green -> rows[0].pixels[1]-green-0
- U2 pad 4: rows[0].pixels[1]-cathode_blue -> rows[0].pixels[1]-blue-0
- U2 pad 6: rows[0].pixels[1]-cathode_cold_white -> rows[0].pixels[1]-cold_white-0
- U3 pad 2: rows[1].pixels[0]-cathode_red -> rows[1].pixels[0]-red-0
- U3 pad 3: rows[1].pixels[0]-cathode_green -> rows[1].pixels[0]-green-0
- U3 pad 4: rows[1].pixels[0]-cathode_blue -> rows[1].pixels[0]-blue-0
- U3 pad 6: rows[1].pixels[0]-cathode_cold_white -> rows[1].pixels[0]-cold_white-0
- U4 pad 2: rows[1].pixels[1]-cathode_red -> rows[1].pixels[1]-red-0
- U4 pad 3: rows[1].pixels[1]-cathode_green -> rows[1].pixels[1]-green-0
- U4 pad 4: rows[1].pixels[1]-cathode_blue -> rows[1].pixels[1]-blue-0
- U4 pad 6: rows[1].pixels[1]-cathode_cold_white -> rows[1].pixels[1]-cold_white-0
Routing:
- net rows[1].pixels[0]-cathode_blue: track 36.2 -> 0.00 mm, vias 2 -> 0
- net rows[0].pixels[1]-cathode_blue: track 36.2 -> 0.00 mm, vias 2 -> 0
- net rows[1].pixels[1]-cathode_blue: track 36.2 -> 0.00 mm, vias 2 -> 0
- net rows[0].pixels[0]-cathode_blue: track 36.2 -> 0.00 mm, vias 2 -> 0
- net rows[0].pixels[0]-anode: track 34.5 -> 0.00 mm
- net rows[1].pixels[1]-anode: track 34.5 -> 3.60 mm
- net rows[0].pixels[1]-anode: track 34.5 -> 3.60 mm
- net rows[1].pixels[0]-anode: track 34.5 -> 3.60 mm
- net rows[0].pixels[0]-cathode_cold_white: track 30.5 -> 0.00 mm, vias 2 -> 0
- net rows[1].pixels[1]-cathode_cold_white: track 30.5 -> 0.00 mm, vias 2 -> 0
- net rows[0].pixels[1]-cathode_cold_white: track 30.5 -> 0.00 mm, vias 2 -> 0
- net rows[1].pixels[0]-cathode_cold_white: track 30.5 -> 0.00 mm, vias 2 -> 0
- net rows[0].pixels[1]-cathode_red: track 24.8 -> 0.00 mm, vias 4 -> 0
- net rows[1].pixels[0]-cathode_red: track 24.8 -> 0.00 mm, vias 4 -> 0
- net rows[0].pixels[0]-cathode_red: track 24.8 -> 0.00 mm, vias 4 -> 0
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
Commit message: broken kicad file
Connections:
- net -red renamed -red-0
- LED1 pad 1: rows[0].pixels[0]-cold_white-1 -> rows[0].pixels[0]-cold_white-0
- LED1 pad 2: -anode -> anode
- LED1 pad 3: rows[0].pixels[0]-blue-1 -> rows[0].pixels[0]-blue-0
- LED1 pad 4: -anode -> anode
- LED1 pad 5: rows[0].pixels[0]-green-1 -> rows[0].pixels[0]-green-0
- LED1 pad 6: -anode -> anode
- LED1 pad 8: -anode -> anode
- LED10 pad 1: rows[1].pixels[0]-cold_white-2 -> rows[1].pixels[0]-cold_white-1
- LED10 pad 2: rows[1].pixels[0]-cold_white-1 -> rows[1].pixels[0]-cold_white-0
- LED10 pad 3: rows[1].pixels[0]-blue-2 -> rows[1].pixels[0]-blue-1
- LED10 pad 4: rows[1].pixels[0]-blue-1 -> rows[1].pixels[0]-blue-0
- LED10 pad 5: rows[1].pixels[0]-green-2 -> rows[1].pixels[0]-green-1
- LED10 pad 6: rows[1].pixels[0]-green-1 -> rows[1].pixels[0]-green-0
- LED10 pad 7: rows[1].pixels[0]-red-2 -> rows[1].pixels[0]-red-1
- LED10 pad 8: rows[1].pixels[0]-red-1 -> rows[1].pixels[0]-red-0
- LED11 pad 1: rows[1].pixels[0]-cold_white-3 -> rows[1].pixels[0]-cold_white-2
- LED11 pad 2: rows[1].pixels[0]-cold_white-2 -> rows[1].pixels[0]-cold_white-1
- LED11 pad 3: rows[1].pixels[0]-blue-3 -> rows[1].pixels[0]-blue-2
- LED11 pad 4: rows[1].pixels[0]-blue-2 -> rows[1].pixels[0]-blue-1
- LED11 pad 5: rows[1].pixels[0]-green-3 -> rows[1].pixels[0]-green-2
- LED11 pad 6: rows[1].pixels[0]-green-2 -> rows[1].pixels[0]-green-1
- LED11 pad 7: rows[1].pixels[0]-red-3 -> rows[1].pixels[0]-red-2
- LED11 pad 8: rows[1].pixels[0]-red-2 -> rows[1].pixels[0]-red-1
- LED12 pad 1: rows[1].pixels[0]-cold_white-0 -> -cold_white-0
- LED12 pad 2: rows[1].pixels[0]-cold_white-3 -> rows[1].pixels[0]-cold_white-2
- LED12 pad 3: rows[1].pixels[0]-blue-0 -> -blue-0
- LED12 pad 4: rows[1].pixels[0]-blue-3 -> rows[1].pixels[0]-blue-2
- LED12 pad 5: rows[1].pixels[0]-green-0 -> -green-3
- LED12 pad 6: rows[1].pixels[0]-green-3 -> rows[1].pixels[0]-green-2
- LED12 pad 7: rows[1].pixels[0]-red-0 -> -red-3
- LED12 pad 8: rows[1].pixels[0]-red-3 -> rows[1].pixels[0]-red-2
- LED13 pad 1: rows[1].pixels[1]-cold_white-1 -> rows[1].pixels[1]-cold_white-0
- LED13 pad 2: rows[1].pixels[1]-anode -> anode
- LED13 pad 3: rows[1].pixels[1]-blue-1 -> rows[1].pixels[1]-blue-0
- LED13 pad 4: rows[1].pixels[1]-anode -> anode
- LED13 pad 5: rows[1].pixels[1]-green-1 -> rows[1].pixels[1]-green-0
- LED13 pad 6: rows[1].pixels[1]-anode -> anode
- LED13 pad 7: rows[1].pixels[1]-red-1 -> rows[1].pixels[1]-red-0
- LED13 pad 8: rows[1].pixels[1]-anode -> anode
- LED14 pad 1: rows[1].pixels[1]-cold_white-2 -> rows[1].pixels[1]-cold_white-1
- LED14 pad 2: rows[1].pixels[1]-cold_white-1 -> rows[1].pixels[1]-cold_white-0
- LED14 pad 3: rows[1].pixels[1]-blue-2 -> rows[1].pixels[1]-blue-1
- LED14 pad 4: rows[1].pixels[1]-blue-1 -> rows[1].pixels[1]-blue-0
- LED14 pad 5: rows[1].pixels[1]-green-2 -> rows[1].pixels[1]-green-1
- LED14 pad 6: rows[1].pixels[1]-green-1 -> rows[1].pixels[1]-green-0
- LED14 pad 7: rows[1].pixels[1]-red-2 -> rows[1].pixels[1]-red-1
- LED14 pad 8: rows[1].pixels[1]-red-1 -> rows[1].pixels[1]-red-0
- LED15 pad 1: rows[1].pixels[1]-cold_white-3 -> rows[1].pixels[1]-cold_white-2
- LED15 pad 2: rows[1].pixels[1]-cold_white-2 -> rows[1].pixels[1]-cold_white-1
- LED15 pad 3: rows[1].pixels[1]-blue-3 -> rows[1].pixels[1]-blue-2
- LED15 pad 4: rows[1].pixels[1]-blue-2 -> rows[1].pixels[1]-blue-1
- LED15 pad 5: rows[1].pixels[1]-green-3 -> rows[1].pixels[1]-green-2
- LED15 pad 6: rows[1].pixels[1]-green-2 -> rows[1].pixels[1]-green-1
- LED15 pad 7: rows[1].pixels[1]-red-3 -> rows[1].pixels[1]-red-2
- LED15 pad 8: rows[1].pixels[1]-red-2 -> rows[1].pixels[1]-red-1
- LED16 pad 1: rows[1].pixels[1]-cold_white-0 -> -cold_white-1
- LED16 pad 2: rows[1].pixels[1]-cold_white-3 -> rows[1].pixels[1]-cold_white-2
- LED16 pad 3: rows[1].pixels[1]-blue-0 -> -blue-1
- LED16 pad 4: rows[1].pixels[1]-blue-3 -> rows[1].pixels[1]-blue-2
- LED16 pad 5: rows[1].pixels[1]-green-0 -> -green-0
- LED16 pad 6: rows[1].pixels[1]-green-3 -> rows[1].pixels[1]-green-2
- LED16 pad 7: rows[1].pixels[1]-red-0 -> -red-1
- LED16 pad 8: rows[1].pixels[1]-red-3 -> rows[1].pixels[1]-red-2
- LED2 pad 1: rows[0].pixels[0]-cold_white-2 -> rows[0].pixels[0]-cold_white-1
- LED2 pad 2: rows[0].pixels[0]-cold_white-1 -> rows[0].pixels[0]-cold_white-0
- LED2 pad 3: rows[0].pixels[0]-blue-2 -> rows[0].pixels[0]-blue-1
- LED2 pad 4: rows[0].pixels[0]-blue-1 -> rows[0].pixels[0]-blue-0
- LED2 pad 5: rows[0].pixels[0]-green-2 -> rows[0].pixels[0]-green-1
- LED2 pad 6: rows[0].pixels[0]-green-1 -> rows[0].pixels[0]-green-0
- LED3 pad 1: rows[0].pixels[0]-cold_white-3 -> rows[0].pixels[0]-cold_white-2
- LED3 pad 2: rows[0].pixels[0]-cold_white-2 -> rows[0].pixels[0]-cold_white-1
- LED3 pad 3: rows[0].pixels[0]-blue-3 -> rows[0].pixels[0]-blue-2
- LED3 pad 4: rows[0].pixels[0]-blue-2 -> rows[0].pixels[0]-blue-1
- LED3 pad 5: rows[0].pixels[0]-green-3 -> rows[0].pixels[0]-green-2
- LED3 pad 6: rows[0].pixels[0]-green-2 -> rows[0].pixels[0]-green-1
- LED4 pad 1: rows[0].pixels[0]-cold_white-0 -> -cold_white-2
- LED4 pad 2: rows[0].pixels[0]-cold_white-3 -> rows[0].pixels[0]-cold_white-2
- LED4 pad 3: rows[0].pixels[0]-blue-0 -> -blue-2
- LED4 pad 4: rows[0].pixels[0]-blue-3 -> rows[0].pixels[0]-blue-2
- LED4 pad 5: rows[0].pixels[0]-green-0 -> -green-1
- LED4 pad 6: rows[0].pixels[0]-green-3 -> rows[0].pixels[0]-green-2
- LED5 pad 1: rows[0].pixels[1]-cold_white-1 -> rows[0].pixels[1]-cold_white-0
- LED5 pad 2: rows[0].pixels[1]-anode -> anode
- LED5 pad 3: rows[0].pixels[1]-blue-1 -> rows[0].pixels[1]-blue-0
- LED5 pad 4: rows[0].pixels[1]-anode -> anode
- LED5 pad 5: rows[0].pixels[1]-green-1 -> rows[0].pixels[1]-green-0
- LED5 pad 6: rows[0].pixels[1]-anode -> anode
- LED5 pad 7: rows[0].pixels[1]-red-1 -> rows[0].pixels[1]-red-0
- LED5 pad 8: rows[0].pixels[1]-anode -> anode
- LED6 pad 1: rows[0].pixels[1]-cold_white-2 -> rows[0].pixels[1]-cold_white-1
- LED6 pad 2: rows[0].pixels[1]-cold_white-1 -> rows[0].pixels[1]-cold_white-0
- LED6 pad 3: rows[0].pixels[1]-blue-2 -> rows[0].pixels[1]-blue-1
- LED6 pad 4: rows[0].pixels[1]-blue-1 -> rows[0].pixels[1]-blue-0
- LED6 pad 5: rows[0].pixels[1]-green-2 -> rows[0].pixels[1]-green-1
- LED6 pad 6: rows[0].pixels[1]-green-1 -> rows[0].pixels[1]-green-0
- LED6 pad 7: rows[0].pixels[1]-red-2 -> rows[0].pixels[1]-red-1
- LED6 pad 8: rows[0].pixels[1]-red-1 -> rows[0].pixels[1]-red-0
- LED7 pad 1: rows[0].pixels[1]-cold_white-3 -> rows[0].pixels[1]-cold_white-2
- LED7 pad 2: rows[0].pixels[1]-cold_white-2 -> rows[0].pixels[1]-cold_white-1
- LED7 pad 3: rows[0].pixels[1]-blue-3 -> rows[0].pixels[1]-blue-2
- LED7 pad 4: rows[0].pixels[1]-blue-2 -> rows[0].pixels[1]-blue-1
- LED7 pad 5: rows[0].pixels[1]-green-3 -> rows[0].pixels[1]-green-2
- LED7 pad 6: rows[0].pixels[1]-green-2 -> rows[0].pixels[1]-green-1
- LED7 pad 7: rows[0].pixels[1]-red-3 -> rows[0].pixels[1]-red-2
- LED7 pad 8: rows[0].pixels[1]-red-2 -> rows[0].pixels[1]-red-1
- LED8 pad 1: rows[0].pixels[1]-cold_white-0 -> -cold_white-3
- LED8 pad 2: rows[0].pixels[1]-cold_white-3 -> rows[0].pixels[1]-cold_white-2
- LED8 pad 3: rows[0].pixels[1]-blue-0 -> -blue-3
- LED8 pad 4: rows[0].pixels[1]-blue-3 -> rows[0].pixels[1]-blue-2
- LED8 pad 5: rows[0].pixels[1]-green-0 -> -green-2
- LED8 pad 6: rows[0].pixels[1]-green-3 -> rows[0].pixels[1]-green-2
- LED8 pad 7: rows[0].pixels[1]-red-0 -> -red-2
- LED8 pad 8: rows[0].pixels[1]-red-3 -> rows[0].pixels[1]-red-2
- LED9 pad 1: rows[1].pixels[0]-cold_white-1 -> rows[1].pixels[0]-cold_white-0
- LED9 pad 2: rows[1].pixels[0]-anode -> anode
- LED9 pad 3: rows[1].pixels[0]-blue-1 -> rows[1].pixels[0]-blue-0
- LED9 pad 4: rows[1].pixels[0]-anode -> anode
- LED9 pad 5: rows[1].pixels[0]-green-1 -> rows[1].pixels[0]-green-0
- LED9 pad 6: rows[1].pixels[0]-anode -> anode
- LED9 pad 7: rows[1].pixels[0]-red-1 -> rows[1].pixels[0]-red-0
- LED9 pad 8: rows[1].pixels[0]-anode -> anode
- U1 pad 1: -anode -> anode
- U1 pad 3: rows[0].pixels[0]-green-0 -> -green-1
- U1 pad 4: rows[0].pixels[0]-blue-0 -> -blue-2
- U1 pad 6: rows[0].pixels[0]-cold_white-0 -> -cold_white-2
- U2 pad 1: rows[0].pixels[1]-anode -> anode
- U2 pad 2: rows[0].pixels[1]-red-0 -> -red-2
- U2 pad 3: rows[0].pixels[1]-green-0 -> -green-2
- U2 pad 4: rows[0].pixels[1]-blue-0 -> -blue-3
- U2 pad 6: rows[0].pixels[1]-cold_white-0 -> -cold_white-3
- U3 pad 1: rows[1].pixels[0]-anode -> anode
- U3 pad 2: rows[1].pixels[0]-red-0 -> -red-3
- U3 pad 3: rows[1].pixels[0]-green-0 -> -green-3
- U3 pad 4: rows[1].pixels[0]-blue-0 -> -blue-0
- U3 pad 6: rows[1].pixels[0]-cold_white-0 -> -cold_white-0
- U4 pad 1: rows[1].pixels[1]-anode -> anode
- U4 pad 2: rows[1].pixels[1]-red-0 -> -red-1
- U4 pad 3: rows[1].pixels[1]-green-0 -> -green-0
- U4 pad 4: rows[1].pixels[1]-blue-0 -> -blue-1
- U4 pad 6: rows[1].pixels[1]-cold_white-0 -> -cold_white-1
- U5 pad 10: OUT5 -> -green-2
- U5 pad 11: OUT6 -> -blue-3
- U5 pad 12: OUT7 -> -cold_white-3
- U5 pad 13: OUT8 -> -red-3
- U5 pad 14: OUT9 -> -green-3
- U5 pad 15: OUT10 -> -blue-0
- U5 pad 16: OUT11 -> -cold_white-0
- U5 pad 17: OUT12 -> -red-1
- U5 pad 18: OUT13 -> -green-0
- U5 pad 19: OUT14 -> -blue-1
- U5 pad 20: OUT15 -> -cold_white-1
- U5 pad 6: OUT1 -> -green-1
- U5 pad 7: OUT2 -> -blue-2
- U5 pad 8: OUT3 -> -cold_white-2
- U5 pad 9: OUT4 -> -red-2
Routing:
- net (no net): track 0.00 -> 27.8 mm
- net rows[1].pixels[1]-cold_white-3: track 7.17 -> 0.00 mm
- net rows[1].pixels[1]-cold_white-2: track 0.00 -> 7.17 mm
- net rows[0].pixels[1]-cold_white-3: track 7.17 -> 0.00 mm
- net rows[0].pixels[1]-cold_white-2: track 0.00 -> 7.17 mm
- net rows[1].pixels[0]-cold_white-3: track 7.17 -> 0.00 mm
- net rows[1].pixels[0]-cold_white-2: track 0.00 -> 7.17 mm
- net rows[0].pixels[0]-cold_white-3: track 7.17 -> 0.00 mm
- net rows[0].pixels[0]-cold_white-2: track 0.00 -> 7.17 mm
- net rows[1].pixels[1]-cold_white-1: track 7.07 -> 0.00 mm
- net rows[1].pixels[1]-cold_white-0: track 0.00 -> 7.07 mm
- net rows[1].pixels[0]-cold_white-1: track 7.07 -> 0.00 mm
- net rows[0].pixels[1]-cold_white-1: track 7.07 -> 0.00 mm
- net rows[0].pixels[1]-cold_white-0: track 0.00 -> 7.07 mm
- net rows[0].pixels[0]-cold_white-1: track 7.07 -> 0.00 mm
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
Commit message: cluster fix up
Parts:
- added C1: 10µF ±10% 25V X5R, Samsung_Electro_Mechanics_CL21A106KAYNNNE:C0805, F.Cu at (6.69, 8.36)
- added C2: 10µF ±10% 25V X5R, Samsung_Electro_Mechanics_CL21A106KAYNNNE:C0805, F.Cu at (8.39, 6.65)
- added C3: 10µF ±10% 25V X5R, Samsung_Electro_Mechanics_CL21A106KAYNNNE:C0805, F.Cu at (6.70, 21.7)
- added C4: 10µF ±10% 25V X5R, Samsung_Electro_Mechanics_CL21A106KAYNNNE:C0805, F.Cu at (23.3, 8.28)
- added C5: 10µF ±10% 25V X5R, Samsung_Electro_Mechanics_CL21A106KAYNNNE:C0805, F.Cu at (21.7, 23.3)
- added C6: 10µF ±10% 25V X5R, Samsung_Electro_Mechanics_CL21A106KAYNNNE:C0805, F.Cu at (8.35, 23.4)
- added C7: 10µF ±10% 25V X5R, Samsung_Electro_Mechanics_CL21A106KAYNNNE:C0805, F.Cu at (23.2, 21.7)
- added C8: 10µF ±10% 25V X5R, Samsung_Electro_Mechanics_CL21A106KAYNNNE:C0805, F.Cu at (21.7, 6.60)
- C9: renamed from C1; moved to B.Cu
- R1: moved to B.Cu
- U1: renamed from U5; moved to B.Cu
- moved C9 29.2 mm to (9.96, 15.0), turned to 90 degrees
- moved R1 29.2 mm to (8.86, 15.0), turned to 90 degrees
- moved U1 29.1 mm to (14.9, 15.0)
- renumbered U1 to U2, U2 to U3, U3 to U4, U4 to U5
Connections:
- LED12 pad 1: -cold_white-0 -> -cold_white-2
- LED12 pad 3: -blue-0 -> -blue-1
- LED12 pad 5: -green-3 -> -green-0
- LED12 pad 7: -red-3 -> -red-0
- LED16 pad 3: -blue-1 -> -blue-0
- LED16 pad 5: -green-0 -> -green-3
- LED16 pad 7: -red-1 -> -red-3
- LED4 pad 1: -cold_white-2 -> -cold_white-0
- LED4 pad 7: -red-0 -> -red-1
- U1 pad 10: -green-2 -> -blue-3
- U1 pad 11: -blue-3 -> -green-2
- U1 pad 12: -cold_white-3 -> -red-2
- U1 pad 16: -cold_white-0 -> -cold_white-1
- U1 pad 17: -red-1 -> -cold_white-2
- U1 pad 18: -green-0 -> -blue-1
- U1 pad 19: -blue-1 -> -green-0
- U1 pad 20: -cold_white-1 -> -red-0
- U1 pad 5: -red-0 -> -cold_white-0
- U1 pad 6: -green-1 -> -blue-2
- U1 pad 7: -blue-2 -> -green-1
- U1 pad 8: -cold_white-2 -> -red-1
- U1 pad 9: -red-2 -> -cold_white-3
Routing:
- net anode: track 0.00 -> 98.5 mm, vias 0 -> 5
- net (no net): track 27.8 -> 0.00 mm
- net -cold_white-2: track 0.00 -> 21.3 mm, vias 0 -> 1
- net -blue-1: track 0.00 -> 19.3 mm, vias 0 -> 1
- net -cold_white-0: track 0.00 -> 17.9 mm, vias 0 -> 1
- net -green-0: track 0.00 -> 17.6 mm, vias 0 -> 1
- net -blue-2: track 0.00 -> 17.3 mm, vias 0 -> 1
- net -green-1: track 0.00 -> 16.9 mm, vias 0 -> 1
- net gnd: track 4.22 -> 20.7 mm, vias 1 -> 5
- net -red-1: track 0.00 -> 16.1 mm, vias 0 -> 1
- net -red-0: track 4.46 -> 15.2 mm, vias 0 -> 1
- net -cold_white-1: track 0.00 -> 10.7 mm, vias 0 -> 1
- net -blue-0: track 0.00 -> 9.39 mm, vias 0 -> 1
- net -green-3: track 0.00 -> 8.66 mm, vias 0 -> 1
- net -red-3: track 0.00 -> 7.86 mm, vias 0 -> 1
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
Commit message: shipped board
Routing:
- net -blue-3: track 6.43 -> 4.48 mm
- net -cold_white-3: track 4.77 -> 4.11 mm

Commit message: built this
Connections:
- C1 pad 2: gnd -> -gnd-1
- C2 pad 2: gnd -> -gnd-1
- C3 pad 2: gnd -> -gnd-1
- C4 pad 2: gnd -> -gnd-1
- C5 pad 2: gnd -> -gnd-1
- C6 pad 2: gnd -> -gnd-1
- C7 pad 2: gnd -> -gnd-1
- C8 pad 2: gnd -> -gnd-1
- C9 pad 2: gnd -> -gnd-0
- R1 pad 2: gnd -> -gnd-0
- U1 pad 1: gnd -> -gnd-0
Routing:
- net gnd: track 20.7 -> 0.00 mm, vias 5 -> 0
- net -gnd-0: track 0.00 -> 20.7 mm, vias 0 -> 5

Commit message: updating rp2040
Connections:
- net -blue-0 renamed rgbs[3]-cathodes-cathode-1
- net -blue-1 renamed rgbs[3]-cathodes-cathode-4
- net -blue-2 renamed rgbs[3]-cathodes-cathode-7
- net -blue-3 renamed rgbs[3]-cathodes-cathode-11
- net -cold_white-0 renamed rgbs[3]-cathodes-cathode-0
- net -cold_white-1 renamed rgbs[3]-cathodes-cathode-2
- net -cold_white-2 renamed rgbs[3]-cathodes-cathode-3
- net -cold_white-3 renamed rgbs[3]-cathodes-cathode-10
- net -gnd-0 renamed power-GND
- net -gnd-1 renamed power_shim-GND
- net -green-0 renamed rgbs[3]-cathodes-cathode-5
- net -green-1 renamed rgbs[3]-cathodes-cathode-8
- net -green-2 renamed rgbs[3]-cathodes-cathode-12
- net -green-3 renamed rgbs[3]-cathodes-cathode-15
- net -red-0 renamed rgbs[3]-cathodes-cathode-6
- net -red-1 renamed rgbs[3]-cathodes-cathode-9
- net -red-2 renamed rgbs[3]-cathodes-cathode-13
- net -red-3 renamed rgbs[3]-cathodes-cathode-14
- net anode renamed power_shim-VCC
- net hv renamed power-VCC
- net rows[0].pixels[0]-blue-0 renamed rgbs[1]-anodes-anode-0
- net rows[0].pixels[0]-blue-1 renamed rgbs[2]-anodes-anode-0
- net rows[0].pixels[0]-blue-2 renamed rgbs[3]-anodes-anode-0
- net rows[0].pixels[0]-cold_white-0 renamed rgbs[1]-anodes-anode-1
- net rows[0].pixels[0]-cold_white-1 renamed rgbs[2]-anodes-anode-1
- net rows[0].pixels[0]-cold_white-2 renamed rgbs[3]-anodes-anode-1
- net rows[0].pixels[0]-green-0 renamed rgbs[1]-anodes-anode-2
- net rows[0].pixels[0]-green-1 renamed rgbs[2]-anodes-anode-2
- net rows[0].pixels[0]-green-2 renamed rgbs[3]-anodes-anode-2
- net rows[0].pixels[0]-red-0 renamed rgbs[1]-anodes-anode-3
- net rows[0].pixels[0]-red-1 renamed rgbs[2]-anodes-anode-3
- net rows[0].pixels[0]-red-2 renamed rgbs[3]-anodes-anode-3
- net rows[0].pixels[1]-blue-0 renamed rgbs[1]-anodes-anode-4
- net rows[0].pixels[1]-blue-1 renamed rgbs[2]-anodes-anode-4
- net rows[0].pixels[1]-blue-2 renamed rgbs[3]-anodes-anode-4
- net rows[0].pixels[1]-cold_white-0 renamed rgbs[1]-anodes-anode-5
- net rows[0].pixels[1]-cold_white-1 renamed rgbs[2]-anodes-anode-5
- net rows[0].pixels[1]-cold_white-2 renamed rgbs[3]-anodes-anode-5
- net rows[0].pixels[1]-green-0 renamed rgbs[1]-anodes-anode-6
- net rows[0].pixels[1]-green-1 renamed rgbs[2]-anodes-anode-6
- net rows[0].pixels[1]-green-2 renamed rgbs[3]-anodes-anode-6
- net rows[0].pixels[1]-red-0 renamed rgbs[1]-anodes-anode-7
- net rows[0].pixels[1]-red-1 renamed rgbs[2]-anodes-anode-7
- net rows[0].pixels[1]-red-2 renamed rgbs[3]-anodes-anode-7
- net rows[1].pixels[0]-blue-0 renamed rgbs[1]-anodes-anode-8
- net rows[1].pixels[0]-blue-1 renamed rgbs[2]-anodes-anode-8
- net rows[1].pixels[0]-blue-2 renamed rgbs[3]-anodes-anode-8
- net rows[1].pixels[0]-cold_white-0 renamed rgbs[1]-anodes-anode-9
- net rows[1].pixels[0]-cold_white-1 renamed rgbs[2]-anodes-anode-9
- net rows[1].pixels[0]-cold_white-2 renamed rgbs[3]-anodes-anode-9
- net rows[1].pixels[0]-green-0 renamed rgbs[1]-anodes-anode-10
- net rows[1].pixels[0]-green-1 renamed rgbs[2]-anodes-anode-10
- net rows[1].pixels[0]-green-2 renamed rgbs[3]-anodes-anode-10
- net rows[1].pixels[0]-red-0 renamed rgbs[1]-anodes-anode-11
- net rows[1].pixels[0]-red-1 renamed rgbs[2]-anodes-anode-11
- net rows[1].pixels[0]-red-2 renamed rgbs[3]-anodes-anode-11
- net rows[1].pixels[1]-blue-0 renamed rgbs[1]-anodes-anode-12
- net rows[1].pixels[1]-blue-1 renamed rgbs[2]-anodes-anode-12
- net rows[1].pixels[1]-blue-2 renamed rgbs[3]-anodes-anode-12
- net rows[1].pixels[1]-cold_white-0 renamed rgbs[1]-anodes-anode-13
- net rows[1].pixels[1]-cold_white-1 renamed rgbs[2]-anodes-anode-13
- net rows[1].pixels[1]-cold_white-2 renamed rgbs[3]-anodes-anode-13
- net rows[1].pixels[1]-green-0 renamed rgbs[1]-anodes-anode-14
- net rows[1].pixels[1]-green-1 renamed rgbs[2]-anodes-anode-14
- net rows[1].pixels[1]-green-2 renamed rgbs[3]-anodes-anode-14
- net rows[1].pixels[1]-red-0 renamed rgbs[1]-anodes-anode-15
- net rows[1].pixels[1]-red-1 renamed rgbs[2]-anodes-anode-15
- net rows[1].pixels[1]-red-2 renamed rgbs[3]-anodes-anode-15

Commit message: tight layout
Routing:
- net power-GND: track 20.7 -> 5.76 mm, vias 5 -> 1
- net power_shim-GND: track 0.00 -> 14.8 mm, vias 0 -> 4
- net rgbs[2]-anodes-anode-13: track 7.07 -> 19.4 mm
- net rgbs[2]-anodes-anode-5: track 7.07 -> 19.4 mm
- net rgbs[2]-anodes-anode-9: track 0.00 -> 12.3 mm
- net rgbs[2]-anodes-anode-1: track 0.00 -> 12.3 mm
- net rgbs[2]-anodes-anode-12: track 5.37 -> 14.9 mm
- net rgbs[3]-anodes-anode-5: track 7.17 -> 12.8 mm
- net rgbs[3]-anodes-anode-1: track 7.17 -> 12.8 mm
- net rgbs[3]-anodes-anode-13: track 7.17 -> 12.8 mm
- net rgbs[3]-anodes-anode-9: track 7.17 -> 12.8 mm
- net rgbs[1]-anodes-anode-1: track 7.07 -> 12.6 mm
- net rgbs[1]-anodes-anode-5: track 7.07 -> 12.6 mm
- net rgbs[1]-anodes-anode-13: track 7.07 -> 12.6 mm
- net rgbs[1]-anodes-anode-9: track 7.07 -> 12.6 mm
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