File: elec/layout/pixel15hl5050/pixel15hl5050.kicad_pcb (KiCad board)
At the start: 2 copper layers, 5 parts

Commit message: pixel refactor
Parts:
- moved LED4 14.9 mm to (-3.70, 3.70), turned to 135 degrees
- moved LED1 11.2 mm to (-3.70, -3.70), turned to 45 degrees
- moved U1 10.6 mm to (-7.50, -7.50)
- moved LED2 10.1 mm to (3.70, -3.70), turned to -45 degrees
- moved LED3 5.35 mm to (3.70, 3.70), turned to -135 degrees
Connections:
- net cathode_ir renamed ir
- net cathode_uv renamed uv
- net cathode_warm_white renamed warm_white
- LED1 pad 1: cathode_cold_white -> -cold_white-1
- LED1 pad 3: cathode_blue -> -blue-1
- LED1 pad 5: cathode_green -> -green-1
- LED1 pad 7: cathode_red -> -red-1
- LED2 pad 1: cathode_cold_white -> -cold_white-2
- LED2 pad 2: anode -> -cold_white-1
- LED2 pad 3: cathode_blue -> -blue-2
- LED2 pad 4: anode -> -blue-1
- LED2 pad 5: cathode_green -> -green-2
- LED2 pad 6: anode -> -green-1
- LED2 pad 7: cathode_red -> -red-2
- LED2 pad 8: anode -> -red-1
- LED3 pad 1: cathode_cold_white -> -cold_white-3
- LED3 pad 2: anode -> -cold_white-2
- LED3 pad 3: cathode_blue -> -blue-3
- LED3 pad 4: anode -> -blue-2
- LED3 pad 5: cathode_green -> -green-3
- LED3 pad 6: anode -> -green-2
- LED3 pad 7: cathode_red -> -red-3
- LED3 pad 8: anode -> -red-2
- LED4 pad 1: cathode_cold_white -> -cold_white-0
- LED4 pad 2: anode -> -cold_white-3
- LED4 pad 3: cathode_blue -> -blue-0
- LED4 pad 4: anode -> -blue-3
- LED4 pad 5: cathode_green -> -green-0
- LED4 pad 6: anode -> -green-3
- LED4 pad 7: cathode_red -> -red-0
- LED4 pad 8: anode -> -red-3
- U1 pad 2: cathode_red -> -red-0
- U1 pad 3: cathode_green -> -green-0
- U1 pad 4: cathode_blue -> -blue-0
- U1 pad 6: cathode_cold_white -> -cold_white-0
Routing:
- net cathode_blue: track 36.2 -> 0.00 mm, vias 2 -> 0
- net anode: track 34.5 -> 3.60 mm
- net cathode_cold_white: track 30.5 -> 0.00 mm, vias 2 -> 0
- net cathode_red: track 24.8 -> 0.00 mm, vias 4 -> 0
- net cathode_green: track 17.7 -> 0.00 mm, vias 2 -> 0
- net -cold_white-3: track 0.00 -> 7.17 mm
- net -cold_white-1: track 0.00 -> 7.07 mm
- net -blue-3: track 0.00 -> 5.54 mm
- net -blue-2: track 0.00 -> 5.37 mm
- net -blue-1: track 0.00 -> 5.37 mm
- net -red-0: track 0.00 -> 4.46 mm
- net -green-3: track 0.00 -> 3.80 mm
- net -green-2: track 0.00 -> 3.74 mm
- net -green-1: track 0.00 -> 3.68 mm
- net -red-3: track 0.00 -> 2.07 mm
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
Commit message: updating rp2040
Connections:
- net -blue-1 renamed rgbs[1]-anodes-anode-0
- net -blue-2 renamed rgbs[2]-anodes-anode-0
- net -blue-3 renamed rgbs[3]-anodes-anode-0
- net -cold_white-1 renamed rgbs[1]-anodes-anode-1
- net -cold_white-2 renamed rgbs[2]-anodes-anode-1
- net -cold_white-3 renamed rgbs[3]-anodes-anode-1
- net -green-1 renamed rgbs[1]-anodes-anode-2
- net -green-2 renamed rgbs[2]-anodes-anode-2
- net -green-3 renamed rgbs[3]-anodes-anode-2
- net -red-1 renamed rgbs[1]-anodes-anode-3
- net -red-2 renamed rgbs[2]-anodes-anode-3
- net -red-3 renamed rgbs[3]-anodes-anode-3
- LED1 pad 2: anode -> rgbs[0]-anodes-anode
- LED1 pad 4: anode -> rgbs[0]-anodes-anode
- LED1 pad 6: anode -> rgbs[0]-anodes-anode
- LED1 pad 8: anode -> rgbs[0]-anodes-anode
- LED4 pad 1: -cold_white-0 -> rgbs[3]-cathodes-cathode-1
- LED4 pad 3: -blue-0 -> rgbs[3]-cathodes-cathode-0
- LED4 pad 5: -green-0 -> rgbs[3]-cathodes-cathode-2
- LED4 pad 7: -red-0 -> rgbs[3]-cathodes-cathode-3
Routing:
- net rgbs[3]-cathodes-cathode-3: track 0.00 -> 4.46 mm
- net -red-0: track 4.46 -> 0.00 mm
- net rgbs[0]-anodes-anode: track 0.00 -> 3.60 mm
- net anode: track 3.60 -> 0.00 mm

Commit message: tight layout
Routing:
- net rgbs[2]-anodes-anode-1: track 0.00 -> 12.3 mm
- net rgbs[3]-anodes-anode-1: track 7.17 -> 12.8 mm
- net rgbs[1]-anodes-anode-1: track 7.07 -> 12.6 mm
- net rgbs[3]-cathodes-cathode-3: track 4.46 -> 0.00 mm
- net rgbs[2]-anodes-anode-0: track 5.37 -> 9.48 mm
- net rgbs[3]-anodes-anode-0: track 5.54 -> 9.49 mm
- net rgbs[1]-anodes-anode-0: track 5.37 -> 9.26 mm
