File: elec/layout/row2/row2.kicad_pcb (KiCad board)
At the start: 2 copper layers, 10 parts

Commit message: cluster with driver
Parts:
- moved LED8 35.7 mm to (18.8, 11.2), turned to 135 degrees
- moved LED4 35.2 mm to (3.80, 11.2), turned to 135 degrees
- moved LED5 33.2 mm to (18.8, 3.80), turned to 45 degrees
- moved LED1 32.8 mm to (3.80, 3.80), turned to 45 degrees
- moved U2 32.7 mm to (15.0, 0.00)
- moved U1 32.3 mm to (0.00, 0.00)
- moved LED6 32.2 mm to (26.2, 3.80), turned to -45 degrees
- moved LED2 31.8 mm to (11.2, 3.80), turned to -45 degrees
- moved LED7 26.9 mm to (26.2, 11.2), turned to -135 degrees
- moved LED3 26.5 mm to (11.2, 11.2), turned to -135 degrees
Connections:
- net pixels[0]-cathode_ir renamed pixels[0]-ir
- net pixels[0]-cathode_uv renamed pixels[0]-uv
- net pixels[0]-cathode_warm_white renamed pixels[0]-warm_white
- net pixels[1]-cathode_ir renamed pixels[1]-ir
- net pixels[1]-cathode_uv renamed pixels[1]-uv
- net pixels[1]-cathode_warm_white renamed pixels[1]-warm_white
- LED1 pad 1: pixels[0]-cathode_cold_white -> pixels[0]-cold_white-1
- LED1 pad 3: pixels[0]-cathode_blue -> pixels[0]-blue-1
- LED1 pad 5: pixels[0]-cathode_green -> pixels[0]-green-1
- LED1 pad 7: pixels[0]-cathode_red -> pixels[0]-red-1
- LED2 pad 1: pixels[0]-cathode_cold_white -> pixels[0]-cold_white-2
- LED2 pad 2: pixels[0]-anode -> pixels[0]-cold_white-1
- LED2 pad 3: pixels[0]-cathode_blue -> pixels[0]-blue-2
- LED2 pad 4: pixels[0]-anode -> pixels[0]-blue-1
- LED2 pad 5: pixels[0]-cathode_green -> pixels[0]-green-2
- LED2 pad 6: pixels[0]-anode -> pixels[0]-green-1
- LED2 pad 7: pixels[0]-cathode_red -> pixels[0]-red-2
- LED2 pad 8: pixels[0]-anode -> pixels[0]-red-1
- LED3 pad 1: pixels[0]-cathode_cold_white -> pixels[0]-cold_white-3
- LED3 pad 2: pixels[0]-anode -> pixels[0]-cold_white-2
- LED3 pad 3: pixels[0]-cathode_blue -> pixels[0]-blue-3
- LED3 pad 4: pixels[0]-anode -> pixels[0]-blue-2
- LED3 pad 5: pixels[0]-cathode_green -> pixels[0]-green-3
- LED3 pad 6: pixels[0]-anode -> pixels[0]-green-2
- LED3 pad 7: pixels[0]-cathode_red -> pixels[0]-red-3
- LED3 pad 8: pixels[0]-anode -> pixels[0]-red-2
- LED4 pad 1: pixels[0]-cathode_cold_white -> pixels[0]-cold_white-0
- LED4 pad 2: pixels[0]-anode -> pixels[0]-cold_white-3
- LED4 pad 3: pixels[0]-cathode_blue -> pixels[0]-blue-0
- LED4 pad 4: pixels[0]-anode -> pixels[0]-blue-3
- LED4 pad 5: pixels[0]-cathode_green -> pixels[0]-green-0
- LED4 pad 6: pixels[0]-anode -> pixels[0]-green-3
- LED4 pad 7: pixels[0]-cathode_red -> pixels[0]-red-0
- LED4 pad 8: pixels[0]-anode -> pixels[0]-red-3
- LED5 pad 1: pixels[1]-cathode_cold_white -> pixels[1]-cold_white-1
- LED5 pad 3: pixels[1]-cathode_blue -> pixels[1]-blue-1
- LED5 pad 5: pixels[1]-cathode_green -> pixels[1]-green-1
- LED5 pad 7: pixels[1]-cathode_red -> pixels[1]-red-1
- LED6 pad 1: pixels[1]-cathode_cold_white -> pixels[1]-cold_white-2
- LED6 pad 2: pixels[1]-anode -> pixels[1]-cold_white-1
- LED6 pad 3: pixels[1]-cathode_blue -> pixels[1]-blue-2
- LED6 pad 4: pixels[1]-anode -> pixels[1]-blue-1
- LED6 pad 5: pixels[1]-cathode_green -> pixels[1]-green-2
- LED6 pad 6: pixels[1]-anode -> pixels[1]-green-1
- LED6 pad 7: pixels[1]-cathode_red -> pixels[1]-red-2
- LED6 pad 8: pixels[1]-anode -> pixels[1]-red-1
- LED7 pad 1: pixels[1]-cathode_cold_white -> pixels[1]-cold_white-3
- LED7 pad 2: pixels[1]-anode -> pixels[1]-cold_white-2
- LED7 pad 3: pixels[1]-cathode_blue -> pixels[1]-blue-3
- LED7 pad 4: pixels[1]-anode -> pixels[1]-blue-2
- LED7 pad 5: pixels[1]-cathode_green -> pixels[1]-green-3
- LED7 pad 6: pixels[1]-anode -> pixels[1]-green-2
- LED7 pad 7: pixels[1]-cathode_red -> pixels[1]-red-3
- LED7 pad 8: pixels[1]-anode -> pixels[1]-red-2
- LED8 pad 1: pixels[1]-cathode_cold_white -> pixels[1]-cold_white-0
- LED8 pad 2: pixels[1]-anode -> pixels[1]-cold_white-3
- LED8 pad 3: pixels[1]-cathode_blue -> pixels[1]-blue-0
- LED8 pad 4: pixels[1]-anode -> pixels[1]-blue-3
- LED8 pad 5: pixels[1]-cathode_green -> pixels[1]-green-0
- LED8 pad 6: pixels[1]-anode -> pixels[1]-green-3
- LED8 pad 7: pixels[1]-cathode_red -> pixels[1]-red-0
- LED8 pad 8: pixels[1]-anode -> pixels[1]-red-3
- U1 pad 2: pixels[0]-cathode_red -> pixels[0]-red-0
- U1 pad 3: pixels[0]-cathode_green -> pixels[0]-green-0
- U1 pad 4: pixels[0]-cathode_blue -> pixels[0]-blue-0
- U1 pad 6: pixels[0]-cathode_cold_white -> pixels[0]-cold_white-0
- U2 pad 2: pixels[1]-cathode_red -> pixels[1]-red-0
- U2 pad 3: pixels[1]-cathode_green -> pixels[1]-green-0
- U2 pad 4: pixels[1]-cathode_blue -> pixels[1]-blue-0
- U2 pad 6: pixels[1]-cathode_cold_white -> pixels[1]-cold_white-0
Routing:
- net pixels[1]-cathode_blue: track 36.2 -> 0.00 mm, vias 2 -> 0
- net pixels[0]-cathode_blue: track 36.2 -> 0.00 mm, vias 2 -> 0
- net pixels[1]-anode: track 34.5 -> 3.60 mm
- net pixels[0]-anode: track 34.5 -> 3.60 mm
- net pixels[0]-cathode_cold_white: track 30.5 -> 0.00 mm, vias 2 -> 0
- net pixels[1]-cathode_cold_white: track 30.5 -> 0.00 mm, vias 2 -> 0
- net pixels[1]-cathode_red: track 24.8 -> 0.00 mm, vias 4 -> 0
- net pixels[0]-cathode_red: track 24.8 -> 0.00 mm, vias 4 -> 0
- net pixels[0]-cathode_green: track 17.7 -> 0.00 mm, vias 2 -> 0
- net pixels[1]-cathode_green: track 17.7 -> 0.00 mm, vias 2 -> 0
- net pixels[1]-cold_white-3: track 0.00 -> 7.17 mm
- net pixels[0]-cold_white-3: track 0.00 -> 7.17 mm
- net pixels[1]-cold_white-1: track 0.00 -> 7.07 mm
- net pixels[0]-cold_white-1: track 0.00 -> 7.07 mm
- net pixels[1]-blue-3: track 0.00 -> 5.54 mm
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
Commit message: updating rp2040
Connections:
- net pixels[0]-blue-1 renamed rgbs[1]-anodes-anode-0
- net pixels[0]-blue-2 renamed rgbs[2]-anodes-anode-0
- net pixels[0]-blue-3 renamed rgbs[3]-anodes-anode-0
- net pixels[0]-cold_white-1 renamed rgbs[1]-anodes-anode-1
- net pixels[0]-cold_white-2 renamed rgbs[2]-anodes-anode-1
- net pixels[0]-cold_white-3 renamed rgbs[3]-anodes-anode-1
- net pixels[0]-green-1 renamed rgbs[1]-anodes-anode-2
- net pixels[0]-green-2 renamed rgbs[2]-anodes-anode-2
- net pixels[0]-green-3 renamed rgbs[3]-anodes-anode-2
- net pixels[0]-red-1 renamed rgbs[1]-anodes-anode-3
- net pixels[0]-red-2 renamed rgbs[2]-anodes-anode-3
- net pixels[0]-red-3 renamed rgbs[3]-anodes-anode-3
- net pixels[1]-blue-1 renamed rgbs[1]-anodes-anode-4
- net pixels[1]-blue-2 renamed rgbs[2]-anodes-anode-4
- net pixels[1]-blue-3 renamed rgbs[3]-anodes-anode-4
- net pixels[1]-cold_white-1 renamed rgbs[1]-anodes-anode-5
- net pixels[1]-cold_white-2 renamed rgbs[2]-anodes-anode-5
- net pixels[1]-cold_white-3 renamed rgbs[3]-anodes-anode-5
- net pixels[1]-green-1 renamed rgbs[1]-anodes-anode-6
- net pixels[1]-green-2 renamed rgbs[2]-anodes-anode-6
- net pixels[1]-green-3 renamed rgbs[3]-anodes-anode-6
- net pixels[1]-red-1 renamed rgbs[1]-anodes-anode-7
- net pixels[1]-red-2 renamed rgbs[2]-anodes-anode-7
- net pixels[1]-red-3 renamed rgbs[3]-anodes-anode-7
- LED1 pad 2: pixels[0]-anode -> rgbs[0]-anodes-anode-0
- LED1 pad 4: pixels[0]-anode -> rgbs[0]-anodes-anode-0
- LED1 pad 6: pixels[0]-anode -> rgbs[0]-anodes-anode-0
- LED1 pad 8: pixels[0]-anode -> rgbs[0]-anodes-anode-0
- LED4 pad 1: pixels[0]-cold_white-0 -> rgbs[3]-cathodes-cathode-1
- LED4 pad 3: pixels[0]-blue-0 -> rgbs[3]-cathodes-cathode-0
- LED4 pad 5: pixels[0]-green-0 -> rgbs[3]-cathodes-cathode-2
- LED4 pad 7: pixels[0]-red-0 -> rgbs[3]-cathodes-cathode-3
- LED5 pad 2: pixels[1]-anode -> rgbs[0]-anodes-anode-1
- LED5 pad 4: pixels[1]-anode -> rgbs[0]-anodes-anode-1
- LED5 pad 6: pixels[1]-anode -> rgbs[0]-anodes-anode-1
- LED5 pad 8: pixels[1]-anode -> rgbs[0]-anodes-anode-1
- LED8 pad 1: pixels[1]-cold_white-0 -> rgbs[3]-cathodes-cathode-5
- LED8 pad 3: pixels[1]-blue-0 -> rgbs[3]-cathodes-cathode-4
- LED8 pad 5: pixels[1]-green-0 -> rgbs[3]-cathodes-cathode-6
- LED8 pad 7: pixels[1]-red-0 -> rgbs[3]-cathodes-cathode-7
Routing:
- net rgbs[3]-cathodes-cathode-7: track 0.00 -> 4.46 mm
- net rgbs[3]-cathodes-cathode-3: track 0.00 -> 4.46 mm
- net pixels[1]-red-0: track 4.46 -> 0.00 mm
- net pixels[0]-red-0: track 4.46 -> 0.00 mm
- net rgbs[0]-anodes-anode-0: track 0.00 -> 3.60 mm
- net pixels[0]-anode: track 3.60 -> 0.00 mm
- net rgbs[0]-anodes-anode-1: track 0.00 -> 3.60 mm
- net pixels[1]-anode: track 3.60 -> 0.00 mm

Commit message: tight layout
Routing:
- net rgbs[2]-anodes-anode-5: track 0.00 -> 12.3 mm
- net rgbs[2]-anodes-anode-1: track 0.00 -> 12.3 mm
- net rgbs[3]-anodes-anode-5: track 7.17 -> 12.8 mm
- net rgbs[3]-anodes-anode-1: track 7.17 -> 12.8 mm
- net rgbs[1]-anodes-anode-5: track 7.07 -> 12.6 mm
- net rgbs[1]-anodes-anode-1: track 7.07 -> 12.6 mm
- net rgbs[3]-cathodes-cathode-7: track 4.46 -> 0.00 mm
- net rgbs[3]-cathodes-cathode-3: track 4.46 -> 0.00 mm
- net rgbs[2]-anodes-anode-4: track 5.37 -> 9.48 mm
- net rgbs[2]-anodes-anode-0: track 5.37 -> 9.48 mm
- net rgbs[3]-anodes-anode-4: track 5.54 -> 9.49 mm
- net rgbs[3]-anodes-anode-0: track 5.54 -> 9.49 mm
- net rgbs[1]-anodes-anode-4: track 5.37 -> 9.26 mm
- net rgbs[1]-anodes-anode-0: track 5.37 -> 9.26 mm
