File: elec/layout/cluster_row/cluster_row.kicad_pcb (KiCad board)
At the start: 2 copper layers, 434 parts

Commit message: wire up cluster row
Connections:
- C1 pad 1: decoupling_capacitors[7]-power_shim-VCC-0 -> power_shim-VCC
- C1 pad 2: decoupling_capacitors[7]-power_shim-GND-0 -> power_shim-GND
- C10 pad 1: decoupling_capacitors[7]-power_shim-VCC-5 -> power_shim-VCC
- C10 pad 2: decoupling_capacitors[7]-power_shim-GND-5 -> power_shim-GND
- C100 pad 1: decoupling_capacitors[7]-power_shim-VCC-2 -> power_shim-VCC
- C100 pad 2: decoupling_capacitors[7]-power_shim-GND-2 -> power_shim-GND
- C101 pad 1: decoupling_capacitors[7]-power_shim-VCC-2 -> power_shim-VCC
- C101 pad 2: decoupling_capacitors[7]-power_shim-GND-2 -> power_shim-GND
- C102 pad 1: decoupling_capacitors[7]-power_shim-VCC-2 -> power_shim-VCC
- C102 pad 2: decoupling_capacitors[7]-power_shim-GND-2 -> power_shim-GND
- C103 pad 1: decoupling_capacitors[7]-power_shim-VCC-2 -> power_shim-VCC
- C103 pad 2: decoupling_capacitors[7]-power_shim-GND-2 -> power_shim-GND
- C104 pad 1: decoupling_capacitors[7]-power_shim-VCC-2 -> power_shim-VCC
- C104 pad 2: decoupling_capacitors[7]-power_shim-GND-2 -> power_shim-GND
- C105 pad 1: decoupling_capacitors[7]-power_shim-VCC-2 -> power_shim-VCC
- C105 pad 2: decoupling_capacitors[7]-power_shim-GND-2 -> power_shim-GND
- C106 pad 1: decoupling_capacitors[7]-power_shim-VCC-2 -> power_shim-VCC
- C106 pad 2: decoupling_capacitors[7]-power_shim-GND-2 -> power_shim-GND
- C107 pad 1: decoupling_capacitors[7]-power_shim-VCC-2 -> power_shim-VCC
- C107 pad 2: decoupling_capacitors[7]-power_shim-GND-2 -> power_shim-GND
- C109 pad 1: decoupling_capacitors[7]-power_shim-VCC-3 -> power_shim-VCC
- C109 pad 2: decoupling_capacitors[7]-power_shim-GND-3 -> power_shim-GND
- C11 pad 1: decoupling_capacitors[7]-power_shim-VCC-5 -> power_shim-VCC
- C11 pad 2: decoupling_capacitors[7]-power_shim-GND-5 -> power_shim-GND
- C110 pad 1: decoupling_capacitors[7]-power_shim-VCC-3 -> power_shim-VCC
- C110 pad 2: decoupling_capacitors[7]-power_shim-GND-3 -> power_shim-GND
- C111 pad 1: decoupling_capacitors[7]-power_shim-VCC-3 -> power_shim-VCC
- C111 pad 2: decoupling_capacitors[7]-power_shim-GND-3 -> power_shim-GND
- C112 pad 1: decoupling_capacitors[7]-power_shim-VCC-3 -> power_shim-VCC
- C112 pad 2: decoupling_capacitors[7]-power_shim-GND-3 -> power_shim-GND
- C113 pad 1: decoupling_capacitors[7]-power_shim-VCC-3 -> power_shim-VCC
- C113 pad 2: decoupling_capacitors[7]-power_shim-GND-3 -> power_shim-GND
- C114 pad 1: decoupling_capacitors[7]-power_shim-VCC-3 -> power_shim-VCC
- C114 pad 2: decoupling_capacitors[7]-power_shim-GND-3 -> power_shim-GND
- C115 pad 1: decoupling_capacitors[7]-power_shim-VCC-3 -> power_shim-VCC
- C115 pad 2: decoupling_capacitors[7]-power_shim-GND-3 -> power_shim-GND
- C116 pad 1: decoupling_capacitors[7]-power_shim-VCC-3 -> power_shim-VCC
- C116 pad 2: decoupling_capacitors[7]-power_shim-GND-3 -> power_shim-GND
- C118 pad 1: decoupling_capacitors[7]-power_shim-VCC-4 -> power_shim-VCC
- C118 pad 2: decoupling_capacitors[7]-power_shim-GND-4 -> power_shim-GND
- C119 pad 1: decoupling_capacitors[7]-power_shim-VCC-4 -> power_shim-VCC
- C119 pad 2: decoupling_capacitors[7]-power_shim-GND-4 -> power_shim-GND
- C12 pad 1: decoupling_capacitors[7]-power_shim-VCC-5 -> power_shim-VCC
- C12 pad 2: decoupling_capacitors[7]-power_shim-GND-5 -> power_shim-GND
- C120 pad 1: decoupling_capacitors[7]-power_shim-VCC-4 -> power_shim-VCC
- C120 pad 2: decoupling_capacitors[7]-power_shim-GND-4 -> power_shim-GND
- C121 pad 1: decoupling_capacitors[7]-power_shim-VCC-4 -> power_shim-VCC
- C121 pad 2: decoupling_capacitors[7]-power_shim-GND-4 -> power_shim-GND
- C122 pad 1: decoupling_capacitors[7]-power_shim-VCC-4 -> power_shim-VCC
- C122 pad 2: decoupling_capacitors[7]-power_shim-GND-4 -> power_shim-GND
- C123 pad 1: decoupling_capacitors[7]-power_shim-VCC-4 -> power_shim-VCC
- C123 pad 2: decoupling_capacitors[7]-power_shim-GND-4 -> power_shim-GND
- C124 pad 1: decoupling_capacitors[7]-power_shim-VCC-4 -> power_shim-VCC
- C124 pad 2: decoupling_capacitors[7]-power_shim-GND-4 -> power_shim-GND
- C125 pad 1: decoupling_capacitors[7]-power_shim-VCC-4 -> power_shim-VCC
- C125 pad 2: decoupling_capacitors[7]-power_shim-GND-4 -> power_shim-GND
- C13 pad 1: decoupling_capacitors[7]-power_shim-VCC-5 -> power_shim-VCC
- C13 pad 2: decoupling_capacitors[7]-power_shim-GND-5 -> power_shim-GND
- C14 pad 1: decoupling_capacitors[7]-power_shim-VCC-5 -> power_shim-VCC
- C14 pad 2: decoupling_capacitors[7]-power_shim-GND-5 -> power_shim-GND
- C15 pad 1: decoupling_capacitors[7]-power_shim-VCC-5 -> power_shim-VCC
- C15 pad 2: decoupling_capacitors[7]-power_shim-GND-5 -> power_shim-GND
- C16 pad 1: decoupling_capacitors[7]-power_shim-VCC-5 -> power_shim-VCC
- C16 pad 2: decoupling_capacitors[7]-power_shim-GND-5 -> power_shim-GND
- C17 pad 1: decoupling_capacitors[7]-power_shim-VCC-5 -> power_shim-VCC
- C17 pad 2: decoupling_capacitors[7]-power_shim-GND-5 -> power_shim-GND
- C19 pad 1: decoupling_capacitors[7]-power_shim-VCC-6 -> power_shim-VCC
- C19 pad 2: decoupling_capacitors[7]-power_shim-GND-6 -> power_shim-GND
- C2 pad 1: decoupling_capacitors[7]-power_shim-VCC-0 -> power_shim-VCC
- C2 pad 2: decoupling_capacitors[7]-power_shim-GND-0 -> power_shim-GND
- C20 pad 1: decoupling_capacitors[7]-power_shim-VCC-6 -> power_shim-VCC
- C20 pad 2: decoupling_capacitors[7]-power_shim-GND-6 -> power_shim-GND
- C21 pad 1: decoupling_capacitors[7]-power_shim-VCC-6 -> power_shim-VCC
- C21 pad 2: decoupling_capacitors[7]-power_shim-GND-6 -> power_shim-GND
- C22 pad 1: decoupling_capacitors[7]-power_shim-VCC-6 -> power_shim-VCC
- C22 pad 2: decoupling_capacitors[7]-power_shim-GND-6 -> power_shim-GND
- C23 pad 1: decoupling_capacitors[7]-power_shim-VCC-6 -> power_shim-VCC
- C23 pad 2: decoupling_capacitors[7]-power_shim-GND-6 -> power_shim-GND
- C24 pad 1: decoupling_capacitors[7]-power_shim-VCC-6 -> power_shim-VCC
- C24 pad 2: decoupling_capacitors[7]-power_shim-GND-6 -> power_shim-GND
- C25 pad 1: decoupling_capacitors[7]-power_shim-VCC-6 -> power_shim-VCC
- C25 pad 2: decoupling_capacitors[7]-power_shim-GND-6 -> power_shim-GND
- C26 pad 1: decoupling_capacitors[7]-power_shim-VCC-6 -> power_shim-VCC
- C26 pad 2: decoupling_capacitors[7]-power_shim-GND-6 -> power_shim-GND
- C28 pad 1: decoupling_capacitors[7]-power_shim-VCC-7 -> power_shim-VCC
- C28 pad 2: decoupling_capacitors[7]-power_shim-GND-7 -> power_shim-GND
- C29 pad 1: decoupling_capacitors[7]-power_shim-VCC-7 -> power_shim-VCC
- C29 pad 2: decoupling_capacitors[7]-power_shim-GND-7 -> power_shim-GND
- C3 pad 1: decoupling_capacitors[7]-power_shim-VCC-0 -> power_shim-VCC
- C3 pad 2: decoupling_capacitors[7]-power_shim-GND-0 -> power_shim-GND
- C30 pad 1: decoupling_capacitors[7]-power_shim-VCC-7 -> power_shim-VCC
- C30 pad 2: decoupling_capacitors[7]-power_shim-GND-7 -> power_shim-GND
- C31 pad 1: decoupling_capacitors[7]-power_shim-VCC-7 -> power_shim-VCC
- C31 pad 2: decoupling_capacitors[7]-power_shim-GND-7 -> power_shim-GND
- C32 pad 1: decoupling_capacitors[7]-power_shim-VCC-7 -> power_shim-VCC
- C32 pad 2: decoupling_capacitors[7]-power_shim-GND-7 -> power_shim-GND
- C33 pad 1: decoupling_capacitors[7]-power_shim-VCC-7 -> power_shim-VCC
- C33 pad 2: decoupling_capacitors[7]-power_shim-GND-7 -> power_shim-GND
- C34 pad 1: decoupling_capacitors[7]-power_shim-VCC-7 -> power_shim-VCC
- C34 pad 2: decoupling_capacitors[7]-power_shim-GND-7 -> power_shim-GND
- C35 pad 1: decoupling_capacitors[7]-power_shim-VCC-7 -> power_shim-VCC
- C35 pad 2: decoupling_capacitors[7]-power_shim-GND-7 -> power_shim-GND
- C37 pad 1: decoupling_capacitors[7]-power_shim-VCC-8 -> power_shim-VCC
- C37 pad 2: decoupling_capacitors[7]-power_shim-GND-8 -> power_shim-GND
- C38 pad 1: decoupling_capacitors[7]-power_shim-VCC-8 -> power_shim-VCC
- C38 pad 2: decoupling_capacitors[7]-power_shim-GND-8 -> power_shim-GND
- C39 pad 1: decoupling_capacitors[7]-power_shim-VCC-8 -> power_shim-VCC
- C39 pad 2: decoupling_capacitors[7]-power_shim-GND-8 -> power_shim-GND
- C4 pad 1: decoupling_capacitors[7]-power_shim-VCC-0 -> power_shim-VCC
- C4 pad 2: decoupling_capacitors[7]-power_shim-GND-0 -> power_shim-GND
- C40 pad 1: decoupling_capacitors[7]-power_shim-VCC-8 -> power_shim-VCC
- C40 pad 2: decoupling_capacitors[7]-power_shim-GND-8 -> power_shim-GND
- C41 pad 1: decoupling_capacitors[7]-power_shim-VCC-8 -> power_shim-VCC
- C41 pad 2: decoupling_capacitors[7]-power_shim-GND-8 -> power_shim-GND
- C42 pad 1: decoupling_capacitors[7]-power_shim-VCC-8 -> power_shim-VCC
- C42 pad 2: decoupling_capacitors[7]-power_shim-GND-8 -> power_shim-GND
- C43 pad 1: decoupling_capacitors[7]-power_shim-VCC-8 -> power_shim-VCC
- C43 pad 2: decoupling_capacitors[7]-power_shim-GND-8 -> power_shim-GND
- C44 pad 1: decoupling_capacitors[7]-power_shim-VCC-8 -> power_shim-VCC
- C44 pad 2: decoupling_capacitors[7]-power_shim-GND-8 -> power_shim-GND
- C46 pad 1: decoupling_capacitors[7]-power_shim-VCC-9 -> power_shim-VCC
- C46 pad 2: decoupling_capacitors[7]-power_shim-GND-9 -> power_shim-GND
- C47 pad 1: decoupling_capacitors[7]-power_shim-VCC-9 -> power_shim-VCC
- C47 pad 2: decoupling_capacitors[7]-power_shim-GND-9 -> power_shim-GND
- C48 pad 1: decoupling_capacitors[7]-power_shim-VCC-9 -> power_shim-VCC
- C48 pad 2: decoupling_capacitors[7]-power_shim-GND-9 -> power_shim-GND
- C49 pad 1: decoupling_capacitors[7]-power_shim-VCC-9 -> power_shim-VCC
- C49 pad 2: decoupling_capacitors[7]-power_shim-GND-9 -> power_shim-GND
- C5 pad 1: decoupling_capacitors[7]-power_shim-VCC-0 -> power_shim-VCC
- C5 pad 2: decoupling_capacitors[7]-power_shim-GND-0 -> power_shim-GND
- C50 pad 1: decoupling_capacitors[7]-power_shim-VCC-9 -> power_shim-VCC
- C50 pad 2: decoupling_capacitors[7]-power_shim-GND-9 -> power_shim-GND
- C51 pad 1: decoupling_capacitors[7]-power_shim-VCC-9 -> power_shim-VCC
- C51 pad 2: decoupling_capacitors[7]-power_shim-GND-9 -> power_shim-GND
- C52 pad 1: decoupling_capacitors[7]-power_shim-VCC-9 -> power_shim-VCC
- C52 pad 2: decoupling_capacitors[7]-power_shim-GND-9 -> power_shim-GND
- C53 pad 1: decoupling_capacitors[7]-power_shim-VCC-9 -> power_shim-VCC
- C53 pad 2: decoupling_capacitors[7]-power_shim-GND-9 -> power_shim-GND
- C55 pad 1: decoupling_capacitors[7]-power_shim-VCC-10 -> power_shim-VCC
- C55 pad 2: decoupling_capacitors[7]-power_shim-GND-10 -> power_shim-GND
- C56 pad 1: decoupling_capacitors[7]-power_shim-VCC-10 -> power_shim-VCC
- C56 pad 2: decoupling_capacitors[7]-power_shim-GND-10 -> power_shim-GND
- C57 pad 1: decoupling_capacitors[7]-power_shim-VCC-10 -> power_shim-VCC
- C57 pad 2: decoupling_capacitors[7]-power_shim-GND-10 -> power_shim-GND
- C58 pad 1: decoupling_capacitors[7]-power_shim-VCC-10 -> power_shim-VCC
- C58 pad 2: decoupling_capacitors[7]-power_shim-GND-10 -> power_shim-GND
- C59 pad 1: decoupling_capacitors[7]-power_shim-VCC-10 -> power_shim-VCC
- C59 pad 2: decoupling_capacitors[7]-power_shim-GND-10 -> power_shim-GND
- C6 pad 1: decoupling_capacitors[7]-power_shim-VCC-0 -> power_shim-VCC
- C6 pad 2: decoupling_capacitors[7]-power_shim-GND-0 -> power_shim-GND
- C60 pad 1: decoupling_capacitors[7]-power_shim-VCC-10 -> power_shim-VCC
- C60 pad 2: decoupling_capacitors[7]-power_shim-GND-10 -> power_shim-GND
- C61 pad 1: decoupling_capacitors[7]-power_shim-VCC-10 -> power_shim-VCC
- C61 pad 2: decoupling_capacitors[7]-power_shim-GND-10 -> power_shim-GND
- C62 pad 1: decoupling_capacitors[7]-power_shim-VCC-10 -> power_shim-VCC
- C62 pad 2: decoupling_capacitors[7]-power_shim-GND-10 -> power_shim-GND
- C64 pad 1: decoupling_capacitors[7]-power_shim-VCC-11 -> power_shim-VCC
- C64 pad 2: decoupling_capacitors[7]-power_shim-GND-11 -> power_shim-GND
- C65 pad 1: decoupling_capacitors[7]-power_shim-VCC-11 -> power_shim-VCC
- C65 pad 2: decoupling_capacitors[7]-power_shim-GND-11 -> power_shim-GND
- C66 pad 1: decoupling_capacitors[7]-power_shim-VCC-11 -> power_shim-VCC
- C66 pad 2: decoupling_capacitors[7]-power_shim-GND-11 -> power_shim-GND
- C67 pad 1: decoupling_capacitors[7]-power_shim-VCC-11 -> power_shim-VCC
- C67 pad 2: decoupling_capacitors[7]-power_shim-GND-11 -> power_shim-GND
- C68 pad 1: decoupling_capacitors[7]-power_shim-VCC-11 -> power_shim-VCC
- C68 pad 2: decoupling_capacitors[7]-power_shim-GND-11 -> power_shim-GND
- C69 pad 1: decoupling_capacitors[7]-power_shim-VCC-11 -> power_shim-VCC
- C69 pad 2: decoupling_capacitors[7]-power_shim-GND-11 -> power_shim-GND
- C7 pad 1: decoupling_capacitors[7]-power_shim-VCC-0 -> power_shim-VCC
- C7 pad 2: decoupling_capacitors[7]-power_shim-GND-0 -> power_shim-GND
- C70 pad 1: decoupling_capacitors[7]-power_shim-VCC-11 -> power_shim-VCC
- C70 pad 2: decoupling_capacitors[7]-power_shim-GND-11 -> power_shim-GND
- C71 pad 1: decoupling_capacitors[7]-power_shim-VCC-11 -> power_shim-VCC
- C71 pad 2: decoupling_capacitors[7]-power_shim-GND-11 -> power_shim-GND
- C73 pad 1: decoupling_capacitors[7]-power_shim-VCC-12 -> power_shim-VCC
- C73 pad 2: decoupling_capacitors[7]-power_shim-GND-12 -> power_shim-GND
- C74 pad 1: decoupling_capacitors[7]-power_shim-VCC-12 -> power_shim-VCC
- C74 pad 2: decoupling_capacitors[7]-power_shim-GND-12 -> power_shim-GND
- C75 pad 1: decoupling_capacitors[7]-power_shim-VCC-12 -> power_shim-VCC
- C75 pad 2: decoupling_capacitors[7]-power_shim-GND-12 -> power_shim-GND
- C76 pad 1: decoupling_capacitors[7]-power_shim-VCC-12 -> power_shim-VCC
- C76 pad 2: decoupling_capacitors[7]-power_shim-GND-12 -> power_shim-GND
- C77 pad 1: decoupling_capacitors[7]-power_shim-VCC-12 -> power_shim-VCC
- C77 pad 2: decoupling_capacitors[7]-power_shim-GND-12 -> power_shim-GND
- C78 pad 1: decoupling_capacitors[7]-power_shim-VCC-12 -> power_shim-VCC
- C78 pad 2: decoupling_capacitors[7]-power_shim-GND-12 -> power_shim-GND
- C79 pad 1: decoupling_capacitors[7]-power_shim-VCC-12 -> power_shim-VCC
- C79 pad 2: decoupling_capacitors[7]-power_shim-GND-12 -> power_shim-GND
- C8 pad 1: decoupling_capacitors[7]-power_shim-VCC-0 -> power_shim-VCC
- C8 pad 2: decoupling_capacitors[7]-power_shim-GND-0 -> power_shim-GND
- C80 pad 1: decoupling_capacitors[7]-power_shim-VCC-12 -> power_shim-VCC
- C80 pad 2: decoupling_capacitors[7]-power_shim-GND-12 -> power_shim-GND
- C82 pad 1: decoupling_capacitors[7]-power_shim-VCC-13 -> power_shim-VCC
- C82 pad 2: decoupling_capacitors[7]-power_shim-GND-13 -> power_shim-GND
- C83 pad 1: decoupling_capacitors[7]-power_shim-VCC-13 -> power_shim-VCC
- C83 pad 2: decoupling_capacitors[7]-power_shim-GND-13 -> power_shim-GND
- C84 pad 1: decoupling_capacitors[7]-power_shim-VCC-13 -> power_shim-VCC
- C84 pad 2: decoupling_capacitors[7]-power_shim-GND-13 -> power_shim-GND
- C85 pad 1: decoupling_capacitors[7]-power_shim-VCC-13 -> power_shim-VCC
- C85 pad 2: decoupling_capacitors[7]-power_shim-GND-13 -> power_shim-GND
- C86 pad 1: decoupling_capacitors[7]-power_shim-VCC-13 -> power_shim-VCC
- C86 pad 2: decoupling_capacitors[7]-power_shim-GND-13 -> power_shim-GND
- C87 pad 1: decoupling_capacitors[7]-power_shim-VCC-13 -> power_shim-VCC
- C87 pad 2: decoupling_capacitors[7]-power_shim-GND-13 -> power_shim-GND
- C88 pad 1: decoupling_capacitors[7]-power_shim-VCC-13 -> power_shim-VCC
- C88 pad 2: decoupling_capacitors[7]-power_shim-GND-13 -> power_shim-GND
- C89 pad 1: decoupling_capacitors[7]-power_shim-VCC-13 -> power_shim-VCC
- C89 pad 2: decoupling_capacitors[7]-power_shim-GND-13 -> power_shim-GND
- C91 pad 1: decoupling_capacitors[7]-power_shim-VCC-1 -> power_shim-VCC
- C91 pad 2: decoupling_capacitors[7]-power_shim-GND-1 -> power_shim-GND
- C92 pad 1: decoupling_capacitors[7]-power_shim-VCC-1 -> power_shim-VCC
- C92 pad 2: decoupling_capacitors[7]-power_shim-GND-1 -> power_shim-GND
- C93 pad 1: decoupling_capacitors[7]-power_shim-VCC-1 -> power_shim-VCC
- C93 pad 2: decoupling_capacitors[7]-power_shim-GND-1 -> power_shim-GND
- C94 pad 1: decoupling_capacitors[7]-power_shim-VCC-1 -> power_shim-VCC
- C94 pad 2: decoupling_capacitors[7]-power_shim-GND-1 -> power_shim-GND
- C95 pad 1: decoupling_capacitors[7]-power_shim-VCC-1 -> power_shim-VCC
- C95 pad 2: decoupling_capacitors[7]-power_shim-GND-1 -> power_shim-GND
- C96 pad 1: decoupling_capacitors[7]-power_shim-VCC-1 -> power_shim-VCC
- C96 pad 2: decoupling_capacitors[7]-power_shim-GND-1 -> power_shim-GND
- C97 pad 1: decoupling_capacitors[7]-power_shim-VCC-1 -> power_shim-VCC
- C97 pad 2: decoupling_capacitors[7]-power_shim-GND-1 -> power_shim-GND
- C98 pad 1: decoupling_capacitors[7]-power_shim-VCC-1 -> power_shim-VCC
- C98 pad 2: decoupling_capacitors[7]-power_shim-GND-1 -> power_shim-GND
- LED1 pad 2: decoupling_capacitors[7]-power_shim-VCC-0 -> power_shim-VCC
- LED1 pad 4: decoupling_capacitors[7]-power_shim-VCC-0 -> power_shim-VCC
- LED1 pad 6: decoupling_capacitors[7]-power_shim-VCC-0 -> power_shim-VCC
- LED1 pad 8: decoupling_capacitors[7]-power_shim-VCC-0 -> power_shim-VCC
- LED101 pad 2: decoupling_capacitors[7]-power_shim-VCC-10 -> power_shim-VCC
- LED101 pad 4: decoupling_capacitors[7]-power_shim-VCC-10 -> power_shim-VCC
- LED101 pad 6: decoupling_capacitors[7]-power_shim-VCC-10 -> power_shim-VCC
- LED101 pad 8: decoupling_capacitors[7]-power_shim-VCC-10 -> power_shim-VCC
- LED105 pad 2: decoupling_capacitors[7]-power_shim-VCC-10 -> power_shim-VCC
- LED105 pad 4: decoupling_capacitors[7]-power_shim-VCC-10 -> power_shim-VCC
- LED105 pad 6: decoupling_capacitors[7]-power_shim-VCC-10 -> power_shim-VCC
- LED105 pad 8: decoupling_capacitors[7]-power_shim-VCC-10 -> power_shim-VCC
- LED109 pad 2: decoupling_capacitors[7]-power_shim-VCC-10 -> power_shim-VCC
- LED109 pad 4: decoupling_capacitors[7]-power_shim-VCC-10 -> power_shim-VCC
- LED109 pad 6: decoupling_capacitors[7]-power_shim-VCC-10 -> power_shim-VCC
- LED109 pad 8: decoupling_capacitors[7]-power_shim-VCC-10 -> power_shim-VCC
- LED113 pad 2: decoupling_capacitors[7]-power_shim-VCC-11 -> power_shim-VCC
- LED113 pad 4: decoupling_capacitors[7]-power_shim-VCC-11 -> power_shim-VCC
- LED113 pad 6: decoupling_capacitors[7]-power_shim-VCC-11 -> power_shim-VCC
- LED113 pad 8: decoupling_capacitors[7]-power_shim-VCC-11 -> power_shim-VCC
- LED117 pad 2: decoupling_capacitors[7]-power_shim-VCC-11 -> power_shim-VCC
- LED117 pad 4: decoupling_capacitors[7]-power_shim-VCC-11 -> power_shim-VCC
- LED117 pad 6: decoupling_capacitors[7]-power_shim-VCC-11 -> power_shim-VCC
- LED117 pad 8: decoupling_capacitors[7]-power_shim-VCC-11 -> power_shim-VCC
- LED121 pad 2: decoupling_capacitors[7]-power_shim-VCC-11 -> power_shim-VCC
- LED121 pad 4: decoupling_capacitors[7]-power_shim-VCC-11 -> power_shim-VCC
- LED121 pad 6: decoupling_capacitors[7]-power_shim-VCC-11 -> power_shim-VCC
- LED121 pad 8: decoupling_capacitors[7]-power_shim-VCC-11 -> power_shim-VCC
- LED125 pad 2: decoupling_capacitors[7]-power_shim-VCC-11 -> power_shim-VCC
- LED125 pad 4: decoupling_capacitors[7]-power_shim-VCC-11 -> power_shim-VCC
- LED125 pad 6: decoupling_capacitors[7]-power_shim-VCC-11 -> power_shim-VCC
- LED125 pad 8: decoupling_capacitors[7]-power_shim-VCC-11 -> power_shim-VCC
- LED129 pad 2: decoupling_capacitors[7]-power_shim-VCC-12 -> power_shim-VCC
- LED129 pad 4: decoupling_capacitors[7]-power_shim-VCC-12 -> power_shim-VCC
- LED129 pad 6: decoupling_capacitors[7]-power_shim-VCC-12 -> power_shim-VCC
- LED129 pad 8: decoupling_capacitors[7]-power_shim-VCC-12 -> power_shim-VCC
- LED13 pad 2: decoupling_capacitors[7]-power_shim-VCC-0 -> power_shim-VCC
- LED13 pad 4: decoupling_capacitors[7]-power_shim-VCC-0 -> power_shim-VCC
- LED13 pad 6: decoupling_capacitors[7]-power_shim-VCC-0 -> power_shim-VCC
- LED13 pad 8: decoupling_capacitors[7]-power_shim-VCC-0 -> power_shim-VCC
- LED133 pad 2: decoupling_capacitors[7]-power_shim-VCC-12 -> power_shim-VCC
- LED133 pad 4: decoupling_capacitors[7]-power_shim-VCC-12 -> power_shim-VCC
- LED133 pad 6: decoupling_capacitors[7]-power_shim-VCC-12 -> power_shim-VCC
- LED133 pad 8: decoupling_capacitors[7]-power_shim-VCC-12 -> power_shim-VCC
- LED137 pad 2: decoupling_capacitors[7]-power_shim-VCC-12 -> power_shim-VCC
- LED137 pad 4: decoupling_capacitors[7]-power_shim-VCC-12 -> power_shim-VCC
- LED137 pad 6: decoupling_capacitors[7]-power_shim-VCC-12 -> power_shim-VCC
- LED137 pad 8: decoupling_capacitors[7]-power_shim-VCC-12 -> power_shim-VCC
- LED141 pad 2: decoupling_capacitors[7]-power_shim-VCC-12 -> power_shim-VCC
- LED141 pad 4: decoupling_capacitors[7]-power_shim-VCC-12 -> power_shim-VCC
- LED141 pad 6: decoupling_capacitors[7]-power_shim-VCC-12 -> power_shim-VCC
- LED141 pad 8: decoupling_capacitors[7]-power_shim-VCC-12 -> power_shim-VCC
- LED145 pad 2: decoupling_capacitors[7]-power_shim-VCC-13 -> power_shim-VCC
- LED145 pad 4: decoupling_capacitors[7]-power_shim-VCC-13 -> power_shim-VCC
- LED145 pad 6: decoupling_capacitors[7]-power_shim-VCC-13 -> power_shim-VCC
- LED145 pad 8: decoupling_capacitors[7]-power_shim-VCC-13 -> power_shim-VCC
- LED149 pad 2: decoupling_capacitors[7]-power_shim-VCC-13 -> power_shim-VCC
- LED149 pad 4: decoupling_capacitors[7]-power_shim-VCC-13 -> power_shim-VCC
- LED149 pad 6: decoupling_capacitors[7]-power_shim-VCC-13 -> power_shim-VCC
- LED149 pad 8: decoupling_capacitors[7]-power_shim-VCC-13 -> power_shim-VCC
- LED153 pad 2: decoupling_capacitors[7]-power_shim-VCC-13 -> power_shim-VCC
- LED153 pad 4: decoupling_capacitors[7]-power_shim-VCC-13 -> power_shim-VCC
- LED153 pad 6: decoupling_capacitors[7]-power_shim-VCC-13 -> power_shim-VCC
- LED153 pad 8: decoupling_capacitors[7]-power_shim-VCC-13 -> power_shim-VCC
- LED157 pad 2: decoupling_capacitors[7]-power_shim-VCC-13 -> power_shim-VCC
- LED157 pad 4: decoupling_capacitors[7]-power_shim-VCC-13 -> power_shim-VCC
- LED157 pad 6: decoupling_capacitors[7]-power_shim-VCC-13 -> power_shim-VCC
- LED157 pad 8: decoupling_capacitors[7]-power_shim-VCC-13 -> power_shim-VCC
- LED161 pad 2: decoupling_capacitors[7]-power_shim-VCC-1 -> power_shim-VCC
- LED161 pad 4: decoupling_capacitors[7]-power_shim-VCC-1 -> power_shim-VCC
- LED161 pad 6: decoupling_capacitors[7]-power_shim-VCC-1 -> power_shim-VCC
- LED161 pad 8: decoupling_capacitors[7]-power_shim-VCC-1 -> power_shim-VCC
- LED165 pad 2: decoupling_capacitors[7]-power_shim-VCC-1 -> power_shim-VCC
- LED165 pad 4: decoupling_capacitors[7]-power_shim-VCC-1 -> power_shim-VCC
- LED165 pad 6: decoupling_capacitors[7]-power_shim-VCC-1 -> power_shim-VCC
- LED165 pad 8: decoupling_capacitors[7]-power_shim-VCC-1 -> power_shim-VCC
- LED169 pad 2: decoupling_capacitors[7]-power_shim-VCC-1 -> power_shim-VCC
- LED169 pad 4: decoupling_capacitors[7]-power_shim-VCC-1 -> power_shim-VCC
- LED169 pad 6: decoupling_capacitors[7]-power_shim-VCC-1 -> power_shim-VCC
- LED169 pad 8: decoupling_capacitors[7]-power_shim-VCC-1 -> power_shim-VCC
- LED17 pad 2: decoupling_capacitors[7]-power_shim-VCC-5 -> power_shim-VCC
- LED17 pad 4: decoupling_capacitors[7]-power_shim-VCC-5 -> power_shim-VCC
- LED17 pad 6: decoupling_capacitors[7]-power_shim-VCC-5 -> power_shim-VCC
- LED17 pad 8: decoupling_capacitors[7]-power_shim-VCC-5 -> power_shim-VCC
- LED173 pad 2: decoupling_capacitors[7]-power_shim-VCC-1 -> power_shim-VCC
- LED173 pad 4: decoupling_capacitors[7]-power_shim-VCC-1 -> power_shim-VCC
- LED173 pad 6: decoupling_capacitors[7]-power_shim-VCC-1 -> power_shim-VCC
- LED173 pad 8: decoupling_capacitors[7]-power_shim-VCC-1 -> power_shim-VCC
- LED177 pad 2: decoupling_capacitors[7]-power_shim-VCC-2 -> power_shim-VCC
- LED177 pad 4: decoupling_capacitors[7]-power_shim-VCC-2 -> power_shim-VCC
- LED177 pad 6: decoupling_capacitors[7]-power_shim-VCC-2 -> power_shim-VCC
- LED177 pad 8: decoupling_capacitors[7]-power_shim-VCC-2 -> power_shim-VCC
- LED181 pad 2: decoupling_capacitors[7]-power_shim-VCC-2 -> power_shim-VCC
- LED181 pad 4: decoupling_capacitors[7]-power_shim-VCC-2 -> power_shim-VCC
- LED181 pad 6: decoupling_capacitors[7]-power_shim-VCC-2 -> power_shim-VCC
- LED181 pad 8: decoupling_capacitors[7]-power_shim-VCC-2 -> power_shim-VCC
- LED185 pad 2: decoupling_capacitors[7]-power_shim-VCC-2 -> power_shim-VCC
- LED185 pad 4: decoupling_capacitors[7]-power_shim-VCC-2 -> power_shim-VCC
- LED185 pad 6: decoupling_capacitors[7]-power_shim-VCC-2 -> power_shim-VCC
- LED185 pad 8: decoupling_capacitors[7]-power_shim-VCC-2 -> power_shim-VCC
- LED189 pad 2: decoupling_capacitors[7]-power_shim-VCC-2 -> power_shim-VCC
- LED189 pad 4: decoupling_capacitors[7]-power_shim-VCC-2 -> power_shim-VCC
- LED189 pad 6: decoupling_capacitors[7]-power_shim-VCC-2 -> power_shim-VCC
- LED189 pad 8: decoupling_capacitors[7]-power_shim-VCC-2 -> power_shim-VCC
- LED193 pad 2: decoupling_capacitors[7]-power_shim-VCC-3 -> power_shim-VCC
- LED193 pad 4: decoupling_capacitors[7]-power_shim-VCC-3 -> power_shim-VCC
- LED193 pad 6: decoupling_capacitors[7]-power_shim-VCC-3 -> power_shim-VCC
- LED193 pad 8: decoupling_capacitors[7]-power_shim-VCC-3 -> power_shim-VCC
- LED197 pad 2: decoupling_capacitors[7]-power_shim-VCC-3 -> power_shim-VCC
- LED197 pad 4: decoupling_capacitors[7]-power_shim-VCC-3 -> power_shim-VCC
- LED197 pad 6: decoupling_capacitors[7]-power_shim-VCC-3 -> power_shim-VCC
- LED197 pad 8: decoupling_capacitors[7]-power_shim-VCC-3 -> power_shim-VCC
- LED201 pad 2: decoupling_capacitors[7]-power_shim-VCC-3 -> power_shim-VCC
- LED201 pad 4: decoupling_capacitors[7]-power_shim-VCC-3 -> power_shim-VCC
- LED201 pad 6: decoupling_capacitors[7]-power_shim-VCC-3 -> power_shim-VCC
- LED201 pad 8: decoupling_capacitors[7]-power_shim-VCC-3 -> power_shim-VCC
- LED205 pad 2: decoupling_capacitors[7]-power_shim-VCC-3 -> power_shim-VCC
- LED205 pad 4: decoupling_capacitors[7]-power_shim-VCC-3 -> power_shim-VCC
- LED205 pad 6: decoupling_capacitors[7]-power_shim-VCC-3 -> power_shim-VCC
- LED205 pad 8: decoupling_capacitors[7]-power_shim-VCC-3 -> power_shim-VCC
- LED209 pad 2: decoupling_capacitors[7]-power_shim-VCC-4 -> power_shim-VCC
- LED209 pad 4: decoupling_capacitors[7]-power_shim-VCC-4 -> power_shim-VCC
- LED209 pad 6: decoupling_capacitors[7]-power_shim-VCC-4 -> power_shim-VCC
- LED209 pad 8: decoupling_capacitors[7]-power_shim-VCC-4 -> power_shim-VCC
- LED21 pad 2: decoupling_capacitors[7]-power_shim-VCC-5 -> power_shim-VCC
- LED21 pad 4: decoupling_capacitors[7]-power_shim-VCC-5 -> power_shim-VCC
- LED21 pad 6: decoupling_capacitors[7]-power_shim-VCC-5 -> power_shim-VCC
- LED21 pad 8: decoupling_capacitors[7]-power_shim-VCC-5 -> power_shim-VCC
- LED213 pad 2: decoupling_capacitors[7]-power_shim-VCC-4 -> power_shim-VCC
- LED213 pad 4: decoupling_capacitors[7]-power_shim-VCC-4 -> power_shim-VCC
- LED213 pad 6: decoupling_capacitors[7]-power_shim-VCC-4 -> power_shim-VCC
- LED213 pad 8: decoupling_capacitors[7]-power_shim-VCC-4 -> power_shim-VCC
- LED217 pad 2: decoupling_capacitors[7]-power_shim-VCC-4 -> power_shim-VCC
- LED217 pad 4: decoupling_capacitors[7]-power_shim-VCC-4 -> power_shim-VCC
- LED217 pad 6: decoupling_capacitors[7]-power_shim-VCC-4 -> power_shim-VCC
- LED217 pad 8: decoupling_capacitors[7]-power_shim-VCC-4 -> power_shim-VCC
- LED221 pad 2: decoupling_capacitors[7]-power_shim-VCC-4 -> power_shim-VCC
- LED221 pad 4: decoupling_capacitors[7]-power_shim-VCC-4 -> power_shim-VCC
- LED221 pad 6: decoupling_capacitors[7]-power_shim-VCC-4 -> power_shim-VCC
- LED221 pad 8: decoupling_capacitors[7]-power_shim-VCC-4 -> power_shim-VCC
- LED25 pad 2: decoupling_capacitors[7]-power_shim-VCC-5 -> power_shim-VCC
- LED25 pad 4: decoupling_capacitors[7]-power_shim-VCC-5 -> power_shim-VCC
- LED25 pad 6: decoupling_capacitors[7]-power_shim-VCC-5 -> power_shim-VCC
- LED25 pad 8: decoupling_capacitors[7]-power_shim-VCC-5 -> power_shim-VCC
- LED29 pad 2: decoupling_capacitors[7]-power_shim-VCC-5 -> power_shim-VCC
- LED29 pad 4: decoupling_capacitors[7]-power_shim-VCC-5 -> power_shim-VCC
- LED29 pad 6: decoupling_capacitors[7]-power_shim-VCC-5 -> power_shim-VCC
- LED29 pad 8: decoupling_capacitors[7]-power_shim-VCC-5 -> power_shim-VCC
- LED33 pad 2: decoupling_capacitors[7]-power_shim-VCC-6 -> power_shim-VCC
- LED33 pad 4: decoupling_capacitors[7]-power_shim-VCC-6 -> power_shim-VCC
- LED33 pad 6: decoupling_capacitors[7]-power_shim-VCC-6 -> power_shim-VCC
- LED33 pad 8: decoupling_capacitors[7]-power_shim-VCC-6 -> power_shim-VCC
- LED37 pad 2: decoupling_capacitors[7]-power_shim-VCC-6 -> power_shim-VCC
- LED37 pad 4: decoupling_capacitors[7]-power_shim-VCC-6 -> power_shim-VCC
- LED37 pad 6: decoupling_capacitors[7]-power_shim-VCC-6 -> power_shim-VCC
- LED37 pad 8: decoupling_capacitors[7]-power_shim-VCC-6 -> power_shim-VCC
- LED41 pad 2: decoupling_capacitors[7]-power_shim-VCC-6 -> power_shim-VCC
- LED41 pad 4: decoupling_capacitors[7]-power_shim-VCC-6 -> power_shim-VCC
- LED41 pad 6: decoupling_capacitors[7]-power_shim-VCC-6 -> power_shim-VCC
- LED41 pad 8: decoupling_capacitors[7]-power_shim-VCC-6 -> power_shim-VCC
- LED45 pad 2: decoupling_capacitors[7]-power_shim-VCC-6 -> power_shim-VCC
- LED45 pad 4: decoupling_capacitors[7]-power_shim-VCC-6 -> power_shim-VCC
- LED45 pad 6: decoupling_capacitors[7]-power_shim-VCC-6 -> power_shim-VCC
- LED45 pad 8: decoupling_capacitors[7]-power_shim-VCC-6 -> power_shim-VCC
- LED49 pad 2: decoupling_capacitors[7]-power_shim-VCC-7 -> power_shim-VCC
- LED49 pad 4: decoupling_capacitors[7]-power_shim-VCC-7 -> power_shim-VCC
- LED49 pad 6: decoupling_capacitors[7]-power_shim-VCC-7 -> power_shim-VCC
- LED49 pad 8: decoupling_capacitors[7]-power_shim-VCC-7 -> power_shim-VCC
- LED5 pad 2: decoupling_capacitors[7]-power_shim-VCC-0 -> power_shim-VCC
- LED5 pad 4: decoupling_capacitors[7]-power_shim-VCC-0 -> power_shim-VCC
- LED5 pad 6: decoupling_capacitors[7]-power_shim-VCC-0 -> power_shim-VCC
- LED5 pad 8: decoupling_capacitors[7]-power_shim-VCC-0 -> power_shim-VCC
- LED53 pad 2: decoupling_capacitors[7]-power_shim-VCC-7 -> power_shim-VCC
- LED53 pad 4: decoupling_capacitors[7]-power_shim-VCC-7 -> power_shim-VCC
- LED53 pad 6: decoupling_capacitors[7]-power_shim-VCC-7 -> power_shim-VCC
- LED53 pad 8: decoupling_capacitors[7]-power_shim-VCC-7 -> power_shim-VCC
- LED57 pad 2: decoupling_capacitors[7]-power_shim-VCC-7 -> power_shim-VCC
- LED57 pad 4: decoupling_capacitors[7]-power_shim-VCC-7 -> power_shim-VCC
- LED57 pad 6: decoupling_capacitors[7]-power_shim-VCC-7 -> power_shim-VCC
- LED57 pad 8: decoupling_capacitors[7]-power_shim-VCC-7 -> power_shim-VCC
- LED61 pad 2: decoupling_capacitors[7]-power_shim-VCC-7 -> power_shim-VCC
- LED61 pad 4: decoupling_capacitors[7]-power_shim-VCC-7 -> power_shim-VCC
- LED61 pad 6: decoupling_capacitors[7]-power_shim-VCC-7 -> power_shim-VCC
- LED61 pad 8: decoupling_capacitors[7]-power_shim-VCC-7 -> power_shim-VCC
- LED65 pad 2: decoupling_capacitors[7]-power_shim-VCC-8 -> power_shim-VCC
- LED65 pad 4: decoupling_capacitors[7]-power_shim-VCC-8 -> power_shim-VCC
- LED65 pad 6: decoupling_capacitors[7]-power_shim-VCC-8 -> power_shim-VCC
- LED65 pad 8: decoupling_capacitors[7]-power_shim-VCC-8 -> power_shim-VCC
- LED69 pad 2: decoupling_capacitors[7]-power_shim-VCC-8 -> power_shim-VCC
- LED69 pad 4: decoupling_capacitors[7]-power_shim-VCC-8 -> power_shim-VCC
- LED69 pad 6: decoupling_capacitors[7]-power_shim-VCC-8 -> power_shim-VCC
- LED69 pad 8: decoupling_capacitors[7]-power_shim-VCC-8 -> power_shim-VCC
- LED73 pad 2: decoupling_capacitors[7]-power_shim-VCC-8 -> power_shim-VCC
- LED73 pad 4: decoupling_capacitors[7]-power_shim-VCC-8 -> power_shim-VCC
- LED73 pad 6: decoupling_capacitors[7]-power_shim-VCC-8 -> power_shim-VCC
- LED73 pad 8: decoupling_capacitors[7]-power_shim-VCC-8 -> power_shim-VCC
- LED77 pad 2: decoupling_capacitors[7]-power_shim-VCC-8 -> power_shim-VCC
- LED77 pad 4: decoupling_capacitors[7]-power_shim-VCC-8 -> power_shim-VCC
- LED77 pad 6: decoupling_capacitors[7]-power_shim-VCC-8 -> power_shim-VCC
- LED77 pad 8: decoupling_capacitors[7]-power_shim-VCC-8 -> power_shim-VCC
- LED81 pad 2: decoupling_capacitors[7]-power_shim-VCC-9 -> power_shim-VCC
- LED81 pad 4: decoupling_capacitors[7]-power_shim-VCC-9 -> power_shim-VCC
- LED81 pad 6: decoupling_capacitors[7]-power_shim-VCC-9 -> power_shim-VCC
- LED81 pad 8: decoupling_capacitors[7]-power_shim-VCC-9 -> power_shim-VCC
- LED85 pad 2: decoupling_capacitors[7]-power_shim-VCC-9 -> power_shim-VCC
- LED85 pad 4: decoupling_capacitors[7]-power_shim-VCC-9 -> power_shim-VCC
- LED85 pad 6: decoupling_capacitors[7]-power_shim-VCC-9 -> power_shim-VCC
- LED85 pad 8: decoupling_capacitors[7]-power_shim-VCC-9 -> power_shim-VCC
- LED89 pad 2: decoupling_capacitors[7]-power_shim-VCC-9 -> power_shim-VCC
- LED89 pad 4: decoupling_capacitors[7]-power_shim-VCC-9 -> power_shim-VCC
- LED89 pad 6: decoupling_capacitors[7]-power_shim-VCC-9 -> power_shim-VCC
- LED89 pad 8: decoupling_capacitors[7]-power_shim-VCC-9 -> power_shim-VCC
- LED9 pad 2: decoupling_capacitors[7]-power_shim-VCC-0 -> power_shim-VCC
- LED9 pad 4: decoupling_capacitors[7]-power_shim-VCC-0 -> power_shim-VCC
- LED9 pad 6: decoupling_capacitors[7]-power_shim-VCC-0 -> power_shim-VCC
- LED9 pad 8: decoupling_capacitors[7]-power_shim-VCC-0 -> power_shim-VCC
- LED93 pad 2: decoupling_capacitors[7]-power_shim-VCC-9 -> power_shim-VCC
- LED93 pad 4: decoupling_capacitors[7]-power_shim-VCC-9 -> power_shim-VCC
- LED93 pad 6: decoupling_capacitors[7]-power_shim-VCC-9 -> power_shim-VCC
- LED93 pad 8: decoupling_capacitors[7]-power_shim-VCC-9 -> power_shim-VCC
- LED97 pad 2: decoupling_capacitors[7]-power_shim-VCC-10 -> power_shim-VCC
- LED97 pad 4: decoupling_capacitors[7]-power_shim-VCC-10 -> power_shim-VCC
- LED97 pad 6: decoupling_capacitors[7]-power_shim-VCC-10 -> power_shim-VCC
- LED97 pad 8: decoupling_capacitors[7]-power_shim-VCC-10 -> power_shim-VCC
- U1 pad 21: driver-gclk-GCLK-0 -> GCLK
- U1 pad 3: driver-dclk-DCLK-0 -> DCLK
- U1 pad 4: driver-le-LE-0 -> LE
- U11 pad 21: driver-gclk-GCLK-6 -> GCLK
- U11 pad 3: driver-dclk-DCLK-6 -> DCLK
- U11 pad 4: driver-le-LE-6 -> LE
- U16 pad 21: driver-gclk-GCLK-7 -> GCLK
- U16 pad 3: driver-dclk-DCLK-7 -> DCLK
- U16 pad 4: driver-le-LE-7 -> LE
- U21 pad 21: driver-gclk-GCLK-8 -> GCLK
- U21 pad 3: driver-dclk-DCLK-8 -> DCLK
- U21 pad 4: driver-le-LE-8 -> LE
- U26 pad 21: driver-gclk-GCLK-9 -> GCLK
- U26 pad 3: driver-dclk-DCLK-9 -> DCLK
- U26 pad 4: driver-le-LE-9 -> LE
- U31 pad 21: driver-gclk-GCLK-10 -> GCLK
- U31 pad 3: driver-dclk-DCLK-10 -> DCLK
- U31 pad 4: driver-le-LE-10 -> LE
- U36 pad 21: driver-gclk-GCLK-11 -> GCLK
- U36 pad 3: driver-dclk-DCLK-11 -> DCLK
- U36 pad 4: driver-le-LE-11 -> LE
- U41 pad 21: driver-gclk-GCLK-12 -> GCLK
- U41 pad 3: driver-dclk-DCLK-12 -> DCLK
- U41 pad 4: driver-le-LE-12 -> LE
- U46 pad 21: driver-gclk-GCLK-13 -> GCLK
- U46 pad 3: driver-dclk-DCLK-13 -> DCLK
- U46 pad 4: driver-le-LE-13 -> LE
- U51 pad 21: driver-gclk-GCLK-1 -> GCLK
- U51 pad 3: driver-dclk-DCLK-1 -> DCLK
- U51 pad 4: driver-le-LE-1 -> LE
- U56 pad 21: driver-gclk-GCLK-2 -> GCLK
- U56 pad 3: driver-dclk-DCLK-2 -> DCLK
- U56 pad 4: driver-le-LE-2 -> LE
- U6 pad 21: driver-gclk-GCLK-5 -> GCLK
- U6 pad 3: driver-dclk-DCLK-5 -> DCLK
- U6 pad 4: driver-le-LE-5 -> LE
- U61 pad 21: driver-gclk-GCLK-3 -> GCLK
- U61 pad 3: driver-dclk-DCLK-3 -> DCLK
- U61 pad 4: driver-le-LE-3 -> LE
- U66 pad 21: driver-gclk-GCLK-4 -> GCLK
- U66 pad 3: driver-dclk-DCLK-4 -> DCLK
- U66 pad 4: driver-le-LE-4 -> LE
Routing:
- net power_shim-VCC: track 0.00 -> 1427.9 mm, vias 0 -> 70
- net DCLK: track 0.00 -> 462.5 mm
- net LE: track 0.00 -> 461.3 mm
- net (no net): track 0.00 -> 159.2 mm, vias 0 -> 42
- net decoupling_capacitors[7]-power_shim-VCC-13: track 102.0 -> 0.00 mm, vias 5 -> 0
- net decoupling_capacitors[7]-power_shim-VCC-11: track 102.0 -> 0.00 mm, vias 5 -> 0
- net decoupling_capacitors[7]-power_shim-VCC-4: track 102.0 -> 0.00 mm, vias 5 -> 0
- net decoupling_capacitors[7]-power_shim-VCC-6: track 102.0 -> 0.00 mm, vias 5 -> 0
- net decoupling_capacitors[7]-power_shim-VCC-0: track 102.0 -> 0.00 mm, vias 5 -> 0
- net decoupling_capacitors[7]-power_shim-VCC-7: track 102.0 -> 0.00 mm, vias 5 -> 0
- net decoupling_capacitors[7]-power_shim-VCC-8: track 102.0 -> 0.00 mm, vias 5 -> 0
- net decoupling_capacitors[7]-power_shim-VCC-5: track 102.0 -> 0.00 mm, vias 5 -> 0
- net decoupling_capacitors[7]-power_shim-VCC-12: track 102.0 -> 0.00 mm, vias 5 -> 0
- net decoupling_capacitors[7]-power_shim-VCC-10: track 102.0 -> 0.00 mm, vias 5 -> 0
- net decoupling_capacitors[7]-power_shim-VCC-3: track 102.0 -> 0.00 mm, vias 5 -> 0
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
Commit message: column and panel layout
Other:
- copper layers 2 -> 32
