File: elec/layout/cluster_row/cluster_row.kicad_pcb (KiCad board)
At the start: 32 copper layers, 434 parts

Commit message: friday checkin
Parts:
- added C127: 100nF ±10% 16V X7R, Samsung_Electro_Mechanics_CL05B104KO5NNNC:C0402, B.Cu at (270.1, 19.2)
- added C128: 100nF ±10% 16V X7R, Samsung_Electro_Mechanics_CL05B104KO5NNNC:C0402, B.Cu at (270.1, 16.8)
- added C129: 100nF ±10% 16V X7R, Samsung_Electro_Mechanics_CL05B104KO5NNNC:C0402, B.Cu at (266.8, 19.2)
- added C130: 100nF ±10% 16V X7R, Samsung_Electro_Mechanics_CL05B104KO5NNNC:C0402, B.Cu at (266.8, 16.8)
- added C131: 100nF ±10% 16V X7R, Samsung_Electro_Mechanics_CL05B104KO5NNNC:C0402, B.Cu at (263.5, 19.2)
- added C132: 100nF ±10% 16V X7R, Samsung_Electro_Mechanics_CL05B104KO5NNNC:C0402, B.Cu at (263.5, 16.8)
- added C133: 100nF ±10% 16V X7R, Samsung_Electro_Mechanics_CL05B104KO5NNNC:C0402, B.Cu at (7.87, 16.1)
- added C134: 100nF ±10% 16V X7R, Samsung_Electro_Mechanics_CL05B104KO5NNNC:C0402, B.Cu at (7.87, 13.8)
- added U71: , Diodes_Incorporated_74LVC1T45DW_7:SC-70-6_L2.2-W1.3-P0.65-LS2.1-BR, B.Cu at (268.5, 18.0)
- added U72: , Diodes_Incorporated_74LVC1T45DW_7:SC-70-6_L2.2-W1.3-P0.65-LS2.1-BR, B.Cu at (265.2, 18.0)
- added U73: , Diodes_Incorporated_74LVC1T45DW_7:SC-70-6_L2.2-W1.3-P0.65-LS2.1-BR, B.Cu at (261.9, 18.0)
- added U74: , Diodes_Incorporated_74LVC1T45DW_7:SC-70-6_L2.2-W1.3-P0.65-LS2.1-BR, B.Cu at (6.24, 14.9)
Connections:
- net power-GND renamed power_b-GND
- net power-VCC renamed power_b-VCC
- U1 pad 2: sdi-line -> signal_b-line
Routing:
- net power_shim-GND: track 48.0 -> 70.7 mm, vias 14 -> 20
- net (no net): track 159.2 -> 136.5 mm, vias 42 -> 36
- net power_b-GND: track 80.6 -> 98.4 mm, vias 14 -> 15
- net LE: track 461.3 -> 472.4 mm, vias 0 -> 2
- net signal_b-line: track 0.00 -> 10.0 mm
- net driver-sdo-line-5: track 0.00 -> 9.52 mm
- net driver-sdo-line-6: track 35.8 -> 27.0 mm
- net DCLK: track 462.5 -> 454.8 mm
- net power_a-VCC: track 0.00 -> 5.21 mm
- net power_b-VCC: track 41.9 -> 47.1 mm
- net rgbs[1]-anodes-anode-77: track 12.6 -> 14.8 mm, vias 0 -> 1
- net rgbs[1]-anodes-anode-78: track 4.01 -> 6.11 mm, vias 0 -> 1
Other:
- copper layers 32 -> 2

Commit message: layout checkin
Parts:
- removed C127, C128, C129, C130, C131, C132, C133, C134: 100nF ±10% 16V X7R, Samsung_Electro_Mechanics_CL05B104KO5NNNC:C0402
- removed U71, U72, U73, U74: , Diodes_Incorporated_74LVC1T45DW_7:SC-70-6_L2.2-W1.3-P0.65-LS2.1-BR
Connections:
- net power_b-GND renamed power-GND
- net power_b-VCC renamed power-VCC
- U1 pad 2: signal_b-line -> sdi-line
Routing:
- net power-VCC: track 47.1 -> 527.0 mm, vias 0 -> 40
- net GCLK: track 0.00 -> 455.2 mm
- net power-GND: track 98.4 -> 80.7 mm, vias 15 -> 14
- net signal_b-line: track 10.0 -> 0.00 mm
- net driver-sdo-line-5: track 9.52 -> 0.67 mm
- net driver-sdo-line-6: track 27.0 -> 35.7 mm
- net DCLK: track 454.8 -> 462.5 mm
- net rgbs[2]-anodes-anode-45: track 19.4 -> 12.1 mm
- net rgbs[2]-anodes-anode-37: track 19.4 -> 12.1 mm
- net rgbs[2]-anodes-anode-165: track 19.4 -> 12.1 mm
- net rgbs[2]-anodes-anode-173: track 19.4 -> 12.1 mm
- net rgbs[2]-anodes-anode-125: track 19.4 -> 12.1 mm
- net rgbs[2]-anodes-anode-117: track 19.4 -> 12.1 mm
- net rgbs[2]-anodes-anode-197: track 19.4 -> 12.1 mm
- net rgbs[2]-anodes-anode-181: track 19.4 -> 12.1 mm
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