File: elec/layout/dual_row/dual_row.kicad_pcb (KiCad board)
At the start: 2 copper layers, 363.4 x 3.6 mm, 882 parts

Commit message: layout checkin
Routing:
- net power_leds-GND: track 143.6 -> 431.5 mm, vias 40 -> 112
- net (no net): track 272.9 -> 0.00 mm, vias 72 -> 0
- net LE: track 1025.0 -> 1004.5 mm
